File: Grbl_Esp32/src/custom/pcb/grbl_shift_register.brd (EAGLE design)
At the start: 10 parts

Commit message: pcb
Parts:
- moved E$6 2.54 mm to (26.7, 77.5)
- moved E$7 1.27 mm to (15.2, 91.4)
- moved E$9 1.27 mm to (19.1, 86.1)
Routing:
- net S$7: track 12.5 -> 9.94 mm
- net S$5: track 36.6 -> 34.3 mm
- net S$9: track 6.88 -> 5.08 mm
- net S$11: track 12.5 -> 11.2 mm
- net S$6: track 42.1 -> 43.0 mm
Changed lines of the file:
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@@
 <layer number="25" name="tNames" color="7" fill="1" visible="no" active="yes"/>
 <layer number="26" name="bNames" color="7" fill="1" visible="yes" active="yes"/>
-<layer number="27" name="tValues" color="7" fill="1" visible="no" active="yes"/>
+<layer number="27" name="tValues" color="7" fill="1" visible="yes" active="yes"/>
 <layer number="28" name="bValues" color="7" fill="1" visible="yes" active="yes"/>
 <layer number="29" name="tStop" color="7" fill="3" visible="no" active="yes"/>
@@
 <attribute name="VALUE" x="10.668" y="66.04" size="1.27" layer="27" ratio="10" rot="R90"/>
 </element>
-<element name="E$6" library="diode" library_urn="urn:adsk.eagle:library:210" package="DO34-7" package3d_urn="urn:adsk.eagle:package:43348/1" value="" x="24.13" y="77.47" rot="R90">
-<attribute name="NAME" x="22.987" y="75.946" size="1.27" layer="25" ratio="10" rot="R90"/>
-<attribute name="VALUE" x="26.543" y="75.946" size="1.27" layer="27" ratio="10" rot="R90"/>
-</element>
-<element name="E$7" library="con-wago-500" library_urn="urn:adsk.eagle:library:195" package="W237-102" package3d_urn="urn:adsk.eagle:package:10688/1" value="" x="15.24" y="90.17">
-<attribute name="NAME" x="11.3938" y="85.1662" size="1.27" layer="25" ratio="10"/>
-<attribute name="VALUE" x="10.2" y="82.55" size="1.27" layer="27" ratio="10"/>
-</element>
-<element name="E$9" library="diode" library_urn="urn:adsk.eagle:library:210" package="DO34-7" package3d_urn="urn:adsk.eagle:package:43348/1" value="" x="19.09413125" y="84.851771875">
-<attribute name="NAME" x="17.57013125" y="85.994771875" size="1.27" layer="25" ratio="10"/>
-<attribute name="VALUE" x="17.57013125" y="82.438771875" size="1.27" layer="27" ratio="10"/>
+<element name="E$6" library="diode" library_urn="urn:adsk.eagle:library:210" package="DO34-7" package3d_urn="urn:adsk.eagle:package:43348/1" value="" x="26.67" y="77.47" rot="R90">
+<attribute name="NAME" x="25.527" y="75.946" size="1.27" layer="25" ratio="10" rot="R90"/>
+<attribute name="VALUE" x="29.083" y="75.946" size="1.27" layer="27" ratio="10" rot="R90"/>
+</element>
+<element name="E$7" library="con-wago-500" library_urn="urn:adsk.eagle:library:195" package="W237-102" package3d_urn="urn:adsk.eagle:package:10688/1" value="" x="15.24" y="91.44">
+<attribute name="NAME" x="11.3938" y="86.4362" size="1.27" layer="25" ratio="10"/>
+<attribute name="VALUE" x="10.2" y="83.82" size="1.27" layer="27" ratio="10"/>
+</element>
+<element name="E$9" library="diode" library_urn="urn:adsk.eagle:library:210" package="DO34-7" package3d_urn="urn:adsk.eagle:package:43348/1" value="" x="19.09413125" y="86.121771875">
+<attribute name="NAME" x="17.57013125" y="87.264771875" size="1.27" layer="25" ratio="10"/>
+<attribute name="VALUE" x="17.57013125" y="83.708771875" size="1.27" layer="27" ratio="10"/>
 </element>
 <element name="E$10" library="diode" library_urn="urn:adsk.eagle:library:210" package="DO34-7" package3d_urn="urn:adsk.eagle:package:43348/1" value="" x="27.94" y="91.44">
@@
 <wire x1="20.32" y1="69.85" x2="19.05" y2="68.58" width="0.8128" layer="16"/>
 <wire x1="16.51" y1="80.01" x2="20.32" y2="80.01" width="0.8128" layer="16"/>
-<wire x1="17.78" y1="83.82" x2="16.51" y2="83.82" width="0.8128" layer="16"/>
-<wire x1="16.51" y1="83.82" x2="15.28413125" y2="82.59413125" width="0.8128" layer="16"/>
-<wire x1="15.24" y1="82.55" x2="15.24" y2="81.28" width="0.8128" layer="16"/>
-<wire x1="15.24" y1="81.28" x2="16.51" y2="80.01" width="0.8128" layer="16"/>
+<wire x1="15.28413125" y1="86.121771875" x2="15.28413125" y2="81.23586875" width="0.8128" layer="16"/>
+<wire x1="15.28413125" y1="81.23586875" x2="16.51" y2="80.01" width="0.8128" layer="16"/>
 <wire x1="20.32" y1="80.01" x2="20.32" y2="69.85" width="0.8128" layer="16"/>
 <contactref element="E$7" pad="1"/>
-<wire x1="12.74" y1="88.9" x2="12.74" y2="85.05" width="0.8128" layer="16"/>
-<wire x1="12.74" y1="85.05" x2="13.97" y2="83.82" width="0.8128" layer="16"/>
 <contactref element="E$9" pad="C"/>
-<wire x1="13.97" y1="83.82" x2="15.24" y2="82.55" width="0.8128" layer="16"/>
-<wire x1="15.28413125" y1="84.851771875" x2="15.28413125" y2="82.59413125" width="0.8128" layer="16"/>
-<wire x1="15.28413125" y1="82.59413125" x2="15.24" y2="82.55" width="0.8128" layer="16"/>
-<wire x1="17.78" y1="83.82" x2="13.97" y2="83.82" width="0.8128" layer="16"/>
+<wire x1="13.97" y1="86.121771875" x2="15.28413125" y2="86.121771875" width="0.8128" layer="16"/>
+<wire x1="17.78" y1="83.82" x2="15.28413125" y2="83.82" width="0.8128" layer="16"/>
+<wire x1="15.28413125" y1="83.82" x2="15.28413125" y2="86.121771875" width="0.8128" layer="16"/>
+<wire x1="12.74" y1="87.351771875" x2="13.97" y2="86.121771875" width="0.8128" layer="16"/>
+<wire x1="12.74" y1="90.17" x2="12.74" y2="87.351771875" width="0.8128" layer="16"/>
 </signal>
 <signal name="S$6">
@@
 <wire x1="22.225" y1="80.645" x2="21.59" y2="81.28" width="0.8128" layer="16"/>
 <contactref element="E$7" pad="2"/>
-<wire x1="20.32" y1="87.63" x2="19.05" y2="88.9" width="0.8128" layer="16"/>
-<wire x1="19.05" y1="88.9" x2="17.74" y2="88.9" width="0.8128" layer="16"/>
+<wire x1="20.955" y1="88.265" x2="19.05" y2="90.17" width="0.8128" layer="16"/>
+<wire x1="19.05" y1="90.17" x2="17.74" y2="90.17" width="0.8128" layer="16"/>
 <wire x1="20.32" y1="81.28" x2="20.32" y2="83.82" width="0.8128" layer="16"/>
 <contactref element="E$10" pad="C"/>
@@
 <wire x1="25.3492" y1="84.912225" x2="24.06954375" y2="83.63256875" width="0.8128" layer="16"/>
 <wire x1="20.50743125" y1="83.63256875" x2="20.32" y2="83.82" width="0.8128" layer="16"/>
-<wire x1="24.13" y1="91.44" x2="20.32" y2="87.63" width="0.8128" layer="16"/>
+<wire x1="24.13" y1="91.44" x2="20.955" y2="88.265" width="0.8128" layer="16"/>
+<wire x1="20.955" y1="88.265" x2="20.32" y2="87.63" width="0.8128" layer="16"/>
 </signal>
 <signal name="S$7">
@@
 <contactref element="E$1" pad="8"/>
 <wire x1="30.48" y1="66.04" x2="29.21" y2="66.04" width="0.8128" layer="16"/>
-<wire x1="29.21" y1="66.04" x2="27.94" y2="67.31" width="0.8128" layer="16"/>
-<wire x1="27.94" y1="72.39" x2="26.67" y2="73.66" width="0.8128" layer="16"/>
-<wire x1="26.67" y1="73.66" x2="24.13" y2="73.66" width="0.8128" layer="16"/>
-<wire x1="27.94" y1="67.31" x2="27.94" y2="72.39" width="0.8128" layer="16"/>
+<wire x1="29.21" y1="66.04" x2="26.67" y2="68.58" width="0.8128" layer="16"/>
+<wire x1="26.67" y1="73.66" x2="26.67" y2="68.58" width="0.8128" layer="16"/>
 </signal>
 <signal name="S$8">
@@
 <contactref element="E$8" pad="1"/>
 <contactref element="E$6" pad="A"/>
-<wire x1="24.13" y1="81.28" x2="25.4" y2="81.28" width="0.8128" layer="16"/>
-<wire x1="25.4" y1="81.28" x2="26.67" y2="82.55" width="0.8128" layer="16"/>
-<wire x1="26.67" y1="82.55" x2="26.67" y2="86.36" width="0.8128" layer="16"/>
+<wire x1="26.67" y1="81.28" x2="26.67" y2="86.36" width="0.8128" layer="16"/>
 </signal>
 <signal name="S$10">
@@
 <contactref element="E$8" pad="4"/>
 <contactref element="E$9" pad="A"/>
-<wire x1="22.90413125" y1="84.851771875" x2="22.90413125" y2="87.67413125" width="0.8128" layer="16"/>
+<wire x1="22.90413125" y1="87.67413125" x2="22.90413125" y2="86.121771875" width="0.8128" layer="16"/>
 <wire x1="26.67" y1="91.44" x2="27.94" y2="91.44" width="0.8128" layer="16"/>
 <wire x1="27.94" y1="91.44" x2="29.21" y2="90.17" width="0.8128" layer="16"/>

Commit message: pcb
Parts:
- added E$11, E$12: (no value), con-lstb:MA06-1
- added E$13: (no value), con-lstb:MA04-1
- moved E$5 1.27 mm to (5.08, 74.9)
Connections:
- new net S$12: E$1.5, E$11.4, E$12.4
- new net S$13: E$1.6, E$11.3, E$12.3
- new net S$14: E$1.7, E$11.2, E$12.2
- new net S$15: E$1.2, E$11.5, E$12.5
- net S$1: now also E$13.4
- net S$2: now also E$13.3
- net S$3: now also E$13.2
- net S$4: now also E$13.1
- net S$7: now also E$11.1, E$12.1
- net S$8: now also E$11.6, E$12.6
Routing:
- net S$15: track 0.00 -> 8.67 mm
- net S$14: track 0.00 -> 8.67 mm
- net S$12: track 0.00 -> 8.67 mm
- net S$8: track 5.08 -> 13.8 mm
- net S$7: track 9.94 -> 18.6 mm
- net S$13: track 0.00 -> 8.67 mm
- net S$3: track 11.3 -> 15.1 mm
- net S$2: track 11.3 -> 15.1 mm
- net S$4: track 12.4 -> 13.6 mm
- net S$1: track 12.4 -> 13.6 mm
- net S$5: track 34.3 -> 35.1 mm
Changed lines of the file:
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@@
 <attribute name="VALUE" x="12.319" y="75.565" size="1.27" layer="27" ratio="10" rot="R90"/>
 </element>
-<element name="E$5" library="con-wago-508" library_urn="urn:adsk.eagle:library:196" package="W237-4P" package3d_urn="urn:adsk.eagle:package:10735/1" value="" x="6.35" y="74.93" rot="R90">
-<attribute name="NAME" x="13.208" y="66.04" size="1.27" layer="25" ratio="10" rot="R90"/>
-<attribute name="VALUE" x="10.668" y="66.04" size="1.27" layer="27" ratio="10" rot="R90"/>
+<element name="E$5" library="con-wago-508" library_urn="urn:adsk.eagle:library:196" package="W237-4P" package3d_urn="urn:adsk.eagle:package:10735/1" value="" x="5.08" y="74.93" rot="R90">
+<attribute name="NAME" x="11.938" y="66.04" size="1.27" layer="25" ratio="10" rot="R90"/>
+<attribute name="VALUE" x="9.398" y="66.04" size="1.27" layer="27" ratio="10" rot="R90"/>
 </element>
 <element name="E$6" library="diode" library_urn="urn:adsk.eagle:library:210" package="DO34-7" package3d_urn="urn:adsk.eagle:package:43348/1" value="" x="26.67" y="77.47" rot="R90">
@@
 <attribute name="NAME" x="25.4" y="90.551" size="1.27" layer="25" ratio="10"/>
 <attribute name="VALUE" x="27.94" y="83.439" size="1.27" layer="27" ratio="10"/>
+</element>
+<element name="E$11" library="con-lstb" library_urn="urn:adsk.eagle:library:162" package="MA06-1" package3d_urn="urn:adsk.eagle:package:8340/1" value="" x="35.56" y="74.93" rot="R90">
+<attribute name="NAME" x="33.909" y="67.31" size="1.27" layer="25" ratio="10" rot="R90"/>
+<attribute name="VALUE" x="38.481" y="72.39" size="1.27" layer="27" ratio="10" rot="R90"/>
+</element>
+<element name="E$12" library="con-lstb" library_urn="urn:adsk.eagle:library:162" package="MA06-1" package3d_urn="urn:adsk.eagle:package:8340/1" value="" x="38.1" y="74.93" rot="R90">
+<attribute name="NAME" x="36.449" y="67.31" size="1.27" layer="25" ratio="10" rot="R90"/>
+<attribute name="VALUE" x="41.021" y="72.39" size="1.27" layer="27" ratio="10" rot="R90"/>
+</element>
+<element name="E$13" library="con-lstb" library_urn="urn:adsk.eagle:library:162" package="MA04-1" package3d_urn="urn:adsk.eagle:package:8337/1" value="" x="11.43" y="74.93" rot="R90">
+<attribute name="NAME" x="9.779" y="69.85" size="1.27" layer="25" ratio="10" rot="R90"/>
+<attribute name="VALUE" x="9.779" y="75.565" size="1.27" layer="27" ratio="10" rot="R90"/>
 </element>
 </elements>
@@
 <contactref element="E$5" pad="4"/>
 <wire x1="17.78" y1="78.74" x2="13.97" y2="78.74" width="0.8128" layer="16"/>
-<wire x1="10.16" y1="82.55" x2="6.985" y2="82.55" width="0.8128" layer="16"/>
-<wire x1="13.97" y1="78.74" x2="10.16" y2="82.55" width="0.8128" layer="16"/>
+<wire x1="7.62" y1="82.55" x2="5.715" y2="82.55" width="0.8128" layer="16"/>
+<contactref element="E$13" pad="4"/>
+<wire x1="13.97" y1="78.74" x2="11.43" y2="78.74" width="0.8128" layer="16"/>
+<wire x1="11.43" y1="78.74" x2="7.62" y2="82.55" width="0.8128" layer="16"/>
 </signal>
 <signal name="S$2">
@@
 <wire x1="13.97" y1="76.2" x2="10.16" y2="76.2" width="0.8128" layer="16"/>
 <wire x1="10.16" y1="76.2" x2="8.89" y2="77.47" width="0.8128" layer="16"/>
-<wire x1="8.89" y1="77.47" x2="6.985" y2="77.47" width="0.8128" layer="16"/>
+<wire x1="8.89" y1="77.47" x2="5.715" y2="77.47" width="0.8128" layer="16"/>
+<contactref element="E$13" pad="3"/>
+<wire x1="11.43" y1="76.2" x2="13.97" y2="76.2" width="0.8128" layer="16"/>
 </signal>
 <signal name="S$3">
@@
 <wire x1="13.97" y1="73.66" x2="10.16" y2="73.66" width="0.8128" layer="16"/>
 <wire x1="10.16" y1="73.66" x2="8.89" y2="72.39" width="0.8128" layer="16"/>
-<wire x1="8.89" y1="72.39" x2="6.985" y2="72.39" width="0.8128" layer="16"/>
+<wire x1="8.89" y1="72.39" x2="5.715" y2="72.39" width="0.8128" layer="16"/>
+<contactref element="E$13" pad="2"/>
+<wire x1="11.43" y1="73.66" x2="13.97" y2="73.66" width="0.8128" layer="16"/>
 </signal>
 <signal name="S$4">
@@
 <contactref element="E$5" pad="1"/>
 <wire x1="17.78" y1="71.12" x2="13.97" y2="71.12" width="0.8128" layer="16"/>
-<wire x1="13.97" y1="71.12" x2="10.16" y2="67.31" width="0.8128" layer="16"/>
-<wire x1="10.16" y1="67.31" x2="6.985" y2="67.31" width="0.8128" layer="16"/>
+<contactref element="E$13" pad="1"/>
+<wire x1="7.62" y1="67.31" x2="5.715" y2="67.31" width="0.8128" layer="16"/>
+<wire x1="11.43" y1="71.12" x2="13.97" y2="71.12" width="0.8128" layer="16"/>
+<wire x1="11.43" y1="71.12" x2="7.62" y2="67.31" width="0.8128" layer="16"/>
 </signal>
 <signal name="S$5">
 <contactref element="E$2" pad="7"/>
 <contactref element="E$2" pad="1"/>
-<wire x1="17.78" y1="68.58" x2="19.05" y2="68.58" width="0.8128" layer="16"/>
-<wire x1="20.32" y1="69.85" x2="19.05" y2="68.58" width="0.8128" layer="16"/>
+<wire x1="17.78" y1="68.58" x2="20.32" y2="68.58" width="0.8128" layer="16"/>
 <wire x1="16.51" y1="80.01" x2="20.32" y2="80.01" width="0.8128" layer="16"/>
 <wire x1="15.28413125" y1="86.121771875" x2="15.28413125" y2="81.23586875" width="0.8128" layer="16"/>
 <wire x1="15.28413125" y1="81.23586875" x2="16.51" y2="80.01" width="0.8128" layer="16"/>
-<wire x1="20.32" y1="80.01" x2="20.32" y2="69.85" width="0.8128" layer="16"/>
+<wire x1="20.32" y1="80.01" x2="20.32" y2="68.58" width="0.8128" layer="16"/>
 <contactref element="E$7" pad="1"/>
 <contactref element="E$9" pad="C"/>
@@
 <contactref element="E$2" pad="2"/>
 <wire x1="30.48" y1="76.2" x2="30.48" y2="78.74" width="0.8128" layer="16"/>
-<wire x1="22.86" y1="78.74" x2="30.48" y2="78.74" width="0.8128" layer="16"/>
+<wire x1="30.48" y1="78.74" x2="22.225" y2="78.74" width="0.8128" layer="16"/>
 <wire x1="21.59" y1="81.28" x2="20.32" y2="81.28" width="0.8128" layer="16"/>
 <wire x1="20.32" y1="81.28" x2="17.78" y2="81.28" width="0.8128" layer="16"/>
-<wire x1="22.86" y1="78.74" x2="22.225" y2="79.375" width="0.8128" layer="16"/>
-<wire x1="22.225" y1="79.375" x2="22.225" y2="80.645" width="0.8128" layer="16"/>
-<wire x1="22.225" y1="80.645" x2="21.59" y2="81.28" width="0.8128" layer="16"/>
+<wire x1="21.59" y1="81.28" x2="22.225" y2="80.645" width="0.8128" layer="16"/>
 <contactref element="E$7" pad="2"/>
 <wire x1="20.955" y1="88.265" x2="19.05" y2="90.17" width="0.8128" layer="16"/>
@@
 <wire x1="24.13" y1="91.44" x2="20.955" y2="88.265" width="0.8128" layer="16"/>
 <wire x1="20.955" y1="88.265" x2="20.32" y2="87.63" width="0.8128" layer="16"/>
+<wire x1="22.225" y1="78.74" x2="22.225" y2="80.645" width="0.8128" layer="16"/>
 </signal>
 <signal name="S$7">
@@
 <wire x1="29.21" y1="66.04" x2="26.67" y2="68.58" width="0.8128" layer="16"/>
 <wire x1="26.67" y1="73.66" x2="26.67" y2="68.58" width="0.8128" layer="16"/>
+<contactref element="E$11" pad="1"/>
+<contactref element="E$12" pad="1"/>
+<wire x1="30.48" y1="66.04" x2="31.75" y2="66.04" width="0.8128" layer="16"/>
+<wire x1="31.75" y1="66.04" x2="34.29" y2="68.58" width="0.8128" layer="16"/>
+<wire x1="34.29" y1="68.58" x2="35.56" y2="68.58" width="0.8128" layer="16"/>
+<wire x1="35.56" y1="68.58" x2="38.1" y2="68.58" width="0.8128" layer="16"/>
 </signal>
 <signal name="S$8">
@@
 <wire x1="30.48" y1="86.36" x2="31.75" y2="86.36" width="0.8128" layer="16"/>
 <wire x1="30.48" y1="83.82" x2="30.48" y2="86.36" width="0.8128" layer="16"/>
+<contactref element="E$11" pad="6"/>
+<contactref element="E$12" pad="6"/>
+<wire x1="30.48" y1="83.82" x2="31.75" y2="83.82" width="0.8128" layer="16"/>
+<wire x1="34.29" y1="81.28" x2="35.56" y2="81.28" width="0.8128" layer="16"/>
+<wire x1="31.75" y1="83.82" x2="34.29" y2="81.28" width="0.8128" layer="16"/>
+<wire x1="35.56" y1="81.28" x2="38.1" y2="81.28" width="0.8128" layer="16"/>
 </signal>
 <signal name="S$9">
@@
 <wire x1="22.90413125" y1="87.67413125" x2="26.67" y2="91.44" width="0.8128" layer="16"/>
 </signal>
+<signal name="S$12">
+<contactref element="E$11" pad="4"/>
+<contactref element="E$1" pad="5"/>
+<contactref element="E$12" pad="4"/>
+<wire x1="30.48" y1="73.66" x2="31.75" y2="73.66" width="0.8128" layer="16"/>
+<wire x1="34.29" y1="76.2" x2="35.56" y2="76.2" width="0.8128" layer="16"/>
+<wire x1="31.75" y1="73.66" x2="34.29" y2="76.2" width="0.8128" layer="16"/>
+<wire x1="35.56" y1="76.2" x2="38.1" y2="76.2" width="0.8128" layer="16"/>
+</signal>
+<signal name="S$13">
+<contactref element="E$11" pad="3"/>
+<contactref element="E$1" pad="6"/>
+<contactref element="E$12" pad="3"/>
+<wire x1="30.48" y1="71.12" x2="31.75" y2="71.12" width="0.8128" layer="16"/>
+<wire x1="31.75" y1="71.12" x2="34.29" y2="73.66" width="0.8128" layer="16"/>
+<wire x1="34.29" y1="73.66" x2="35.56" y2="73.66" width="0.8128" layer="16"/>
+<wire x1="35.56" y1="73.66" x2="38.1" y2="73.66" width="0.8128" layer="16"/>
+</signal>
+<signal name="S$14">
+<contactref element="E$11" pad="2"/>
+<contactref element="E$1" pad="7"/>
+<contactref element="E$12" pad="2"/>
+<wire x1="30.48" y1="68.58" x2="31.75" y2="68.58" width="0.8128" layer="16"/>
+<wire x1="31.75" y1="68.58" x2="34.29" y2="71.12" width="0.8128" layer="16"/>
+<wire x1="34.29" y1="71.12" x2="35.56" y2="71.12" width="0.8128" layer="16"/>
+<wire x1="35.56" y1="71.12" x2="38.1" y2="71.12" width="0.8128" layer="16"/>
+</signal>
+<signal name="S$15">
+<contactref element="E$11" pad="5"/>
+<contactref element="E$1" pad="2"/>
+<contactref element="E$12" pad="5"/>
+<wire x1="30.48" y1="81.28" x2="31.75" y2="81.28" width="0.8128" layer="16"/>
+<wire x1="31.75" y1="81.28" x2="34.29" y2="78.74" width="0.8128" layer="16"/>
+<wire x1="34.29" y1="78.74" x2="35.56" y2="78.74" width="0.8128" layer="16"/>
+<wire x1="35.56" y1="78.74" x2="38.1" y2="78.74" width="0.8128" layer="16"/>
+</signal>
 </signals>

Commit message: pcb
Parts:
- moved E$5 1.27 mm to (3.81, 74.9)
Routing:
- net S$4: track 13.6 -> 14.9 mm
- net S$3: track 15.1 -> 16.4 mm
- net S$2: track 15.1 -> 16.4 mm
- net S$1: track 13.6 -> 14.9 mm
Changed lines of the file:
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@@
 <attribute name="VALUE" x="12.319" y="75.565" size="1.27" layer="27" ratio="10" rot="R90"/>
 </element>
-<element name="E$5" library="con-wago-508" library_urn="urn:adsk.eagle:library:196" package="W237-4P" package3d_urn="urn:adsk.eagle:package:10735/1" value="" x="5.08" y="74.93" rot="R90">
-<attribute name="NAME" x="11.938" y="66.04" size="1.27" layer="25" ratio="10" rot="R90"/>
-<attribute name="VALUE" x="9.398" y="66.04" size="1.27" layer="27" ratio="10" rot="R90"/>
+<element name="E$5" library="con-wago-508" library_urn="urn:adsk.eagle:library:196" package="W237-4P" package3d_urn="urn:adsk.eagle:package:10735/1" value="" x="3.81" y="74.93" rot="R90">
+<attribute name="NAME" x="10.668" y="66.04" size="1.27" layer="25" ratio="10" rot="R90"/>
+<attribute name="VALUE" x="8.128" y="66.04" size="1.27" layer="27" ratio="10" rot="R90"/>
 </element>
 <element name="E$6" library="diode" library_urn="urn:adsk.eagle:library:210" package="DO34-7" package3d_urn="urn:adsk.eagle:package:43348/1" value="" x="26.67" y="77.47" rot="R90">
@@
 <contactref element="E$5" pad="4"/>
 <wire x1="17.78" y1="78.74" x2="13.97" y2="78.74" width="0.8128" layer="16"/>
-<wire x1="7.62" y1="82.55" x2="5.715" y2="82.55" width="0.8128" layer="16"/>
+<wire x1="7.62" y1="82.55" x2="4.445" y2="82.55" width="0.8128" layer="16"/>
 <contactref element="E$13" pad="4"/>
 <wire x1="13.97" y1="78.74" x2="11.43" y2="78.74" width="0.8128" layer="16"/>
@@
 <wire x1="13.97" y1="76.2" x2="10.16" y2="76.2" width="0.8128" layer="16"/>
 <wire x1="10.16" y1="76.2" x2="8.89" y2="77.47" width="0.8128" layer="16"/>
-<wire x1="8.89" y1="77.47" x2="5.715" y2="77.47" width="0.8128" layer="16"/>
+<wire x1="8.89" y1="77.47" x2="4.445" y2="77.47" width="0.8128" layer="16"/>
 <contactref element="E$13" pad="3"/>
 <wire x1="11.43" y1="76.2" x2="13.97" y2="76.2" width="0.8128" layer="16"/>
@@
 <wire x1="13.97" y1="73.66" x2="10.16" y2="73.66" width="0.8128" layer="16"/>
 <wire x1="10.16" y1="73.66" x2="8.89" y2="72.39" width="0.8128" layer="16"/>
-<wire x1="8.89" y1="72.39" x2="5.715" y2="72.39" width="0.8128" layer="16"/>
+<wire x1="8.89" y1="72.39" x2="4.445" y2="72.39" width="0.8128" layer="16"/>
 <contactref element="E$13" pad="2"/>
 <wire x1="11.43" y1="73.66" x2="13.97" y2="73.66" width="0.8128" layer="16"/>
@@
 <wire x1="17.78" y1="71.12" x2="13.97" y2="71.12" width="0.8128" layer="16"/>
 <contactref element="E$13" pad="1"/>
-<wire x1="7.62" y1="67.31" x2="5.715" y2="67.31" width="0.8128" layer="16"/>
+<wire x1="7.62" y1="67.31" x2="4.445" y2="67.31" width="0.8128" layer="16"/>
 <wire x1="11.43" y1="71.12" x2="13.97" y2="71.12" width="0.8128" layer="16"/>
 <wire x1="11.43" y1="71.12" x2="7.62" y2="67.31" width="0.8128" layer="16"/>
@@
 <contactref element="E$2" pad="1"/>
 <wire x1="17.78" y1="68.58" x2="20.32" y2="68.58" width="0.8128" layer="16"/>
-<wire x1="16.51" y1="80.01" x2="20.32" y2="80.01" width="0.8128" layer="16"/>
+<wire x1="16.51" y1="80.01" x2="20.32" y2="80.01" width="0.6096" layer="16"/>
 <wire x1="15.28413125" y1="86.121771875" x2="15.28413125" y2="81.23586875" width="0.8128" layer="16"/>
-<wire x1="15.28413125" y1="81.23586875" x2="16.51" y2="80.01" width="0.8128" layer="16"/>
+<wire x1="15.28413125" y1="81.23586875" x2="16.51" y2="80.01" width="0.6096" layer="16"/>
 <wire x1="20.32" y1="80.01" x2="20.32" y2="68.58" width="0.8128" layer="16"/>
 <contactref element="E$7" pad="1"/>
@@
 <contactref element="E$8" pad="2"/>
 <wire x1="26.67" y1="88.9" x2="25.3492" y2="87.5792" width="0.8128" layer="16"/>
-<wire x1="25.3492" y1="87.5792" x2="25.3492" y2="84.912225" width="0.8128" layer="16"/>
+<wire x1="25.3492" y1="87.5792" x2="25.3492" y2="84.912225" width="0.6096" layer="16"/>
 <wire x1="24.06954375" y1="83.63256875" x2="20.50743125" y2="83.63256875" width="0.8128" layer="16"/>
 <wire x1="25.3492" y1="84.912225" x2="24.06954375" y2="83.63256875" width="0.8128" layer="16"/>
@@
 <wire x1="27.94" y1="91.44" x2="29.21" y2="90.17" width="0.8128" layer="16"/>
 <wire x1="29.21" y1="90.17" x2="29.21" y2="88.9" width="0.8128" layer="16"/>
-<wire x1="22.90413125" y1="87.67413125" x2="26.67" y2="91.44" width="0.8128" layer="16"/>
+<wire x1="22.90413125" y1="87.67413125" x2="26.67" y2="91.44" width="0.6096" layer="16"/>
 </signal>
 <signal name="S$12">
