File: Grbl_Esp32/src/custom/pcb/grbl_shift_register.brd (EAGLE design)
At the start: 13 parts

Commit message: pcb
Parts:
- added E$14, E$25, E$26, E$37, E$38: (no value), con-lsta:FE08
- added E$15, E$24, E$27, E$36, E$39, E$48: (no value), con-lstb:MA04-1
- added E$16, E$28, E$40: (no value), con-wago-508:W237-4P
- added E$17, E$19, E$20, E$29, E$31, E$32, E$41, E$43, E$44: (no value), diode:DO34-7
- added E$18, E$30, E$42: (no value), con-wago-500:W237-102
- added E$21, E$33, E$45: (no value), con-lstb:MA03-2
- added E$22, E$23, E$34, E$35, E$46, E$47: (no value), con-lstb:MA06-1
- moved E$3 9.16 mm to (30.5, 45.7), turned to 270 degrees
Connections:
- new net S$16: E$14.3, E$15.4, E$16.4, E$24.4
- new net S$17: E$14.4, E$15.3, E$16.3, E$24.3
- new net S$18: E$14.5, E$15.2, E$16.2, E$24.2
- new net S$19: E$14.6, E$15.1, E$16.1, E$24.1
- new net S$20: E$26.3, E$27.4, E$28.4, E$36.4
- new net S$21: E$26.4, E$27.3, E$28.3, E$36.3
- new net S$22: E$17.C, E$22.1, E$23.1, E$3.8
- new net S$23: E$21.3, E$21.5, E$22.6, E$23.6, E$3.1
- new net S$24: E$17.A, E$21.1
- new net S$25: E$20.A, E$21.6
- new net S$26: E$19.A, E$21.4
- new net S$27: E$22.4, E$23.4, E$3.5
- new net S$28: E$22.3, E$23.3, E$3.6
- new net S$29: E$22.2, E$23.2, E$3.7
- new net S$30: E$22.5, E$23.5, E$3.2
- new net S$31: E$26.5, E$27.2, E$28.2, E$36.2
- new net S$32: E$26.6, E$27.1, E$28.1, E$36.1
- new net S$33: E$26.1, E$26.7, E$30.1, E$31.C, E$38.1, E$38.7, E$42.1, E$43.C
- new net S$34: E$25.3, E$25.4, E$26.2, E$30.2, E$32.C, E$33.2, E$37.3, E$37.4, E$38.2, E$42.2, E$44.C, E$45.2
- new net S$35: E$25.8, E$29.C, E$34.1, E$35.1
- new net S$36: E$25.1, E$33.3, E$33.5, E$34.6, E$35.6
- new net S$37: E$29.A, E$33.1
- new net S$38: E$32.A, E$33.6
- new net S$39: E$31.A, E$33.4
- new net S$40: E$25.5, E$34.4, E$35.4
- new net S$41: E$25.6, E$34.3, E$35.3
- new net S$42: E$25.7, E$34.2, E$35.2
- new net S$43: E$25.2, E$34.5, E$35.5
- new net S$44: E$38.3, E$39.4, E$40.4, E$48.4
- new net S$45: E$38.4, E$39.3, E$40.3, E$48.3
- new net S$46: E$38.5, E$39.2, E$40.2, E$48.2
- new net S$47: E$38.6, E$39.1, E$40.1, E$48.1
- new net S$48: E$37.8, E$41.C, E$46.1, E$47.1
- new net S$49: E$37.1, E$45.3, E$45.5, E$46.6, E$47.6
- new net S$50: E$41.A, E$45.1
- new net S$51: E$44.A, E$45.6
- new net S$52: E$43.A, E$45.4
- new net S$53: E$37.5, E$46.4, E$47.4
- new net S$54: E$37.6, E$46.3, E$47.3
- new net S$55: E$37.7, E$46.2, E$47.2
- new net S$56: E$37.2, E$46.5, E$47.5
- net S$5: now also E$14.1, E$14.7, E$18.1, E$19.C
- net S$6: now also E$14.2, E$18.2, E$20.C, E$21.2, E$3.3, E$3.4
Routing:
- net S$34: track 0.00 -> 103.2 mm
- net S$33: track 0.00 -> 83.1 mm
- net S$6: track 43.3 -> 103.2 mm
- net S$5: track 35.1 -> 83.1 mm
- net S$35: track 0.00 -> 18.6 mm
- net S$22: track 0.00 -> 18.6 mm
- net S$48: track 0.00 -> 18.6 mm
- net S$18: track 0.00 -> 16.4 mm
- net S$46: track 0.00 -> 16.4 mm
- net S$45: track 0.00 -> 16.4 mm
- net S$31: track 0.00 -> 16.4 mm
- net S$21: track 0.00 -> 16.4 mm
- net S$17: track 0.00 -> 16.4 mm
- net S$44: track 0.00 -> 14.9 mm
- net S$16: track 0.00 -> 14.9 mm
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
Commit message: pcb
Connections:
- removed net S$33: E$26.1, E$26.7, E$30.1, E$31.C, E$38.1, E$38.7, E$42.1, E$43.C
- removed net S$34: E$25.3, E$25.4, E$26.2, E$30.2, E$32.C, E$33.2, E$37.3, E$37.4, E$38.2, E$42.2, E$44.C, E$45.2
- net S$5: now also E$26.1, E$26.7, E$30.1, E$31.C, E$38.1, E$38.7, E$42.1, E$43.C
- net S$6: now also E$25.3, E$25.4, E$26.2, E$30.2, E$32.C, E$33.2, E$37.3, E$37.4, E$38.2, E$42.2, E$44.C, E$45.2
Routing:
- net S$6: track 103.2 -> 222.8 mm
- net S$34: track 103.2 -> 0.00 mm
- net S$5: track 83.1 -> 179.2 mm
- net S$33: track 83.1 -> 0.00 mm

Commit message: pcb
Parts:
- added E$49, E$50, E$61, E$62: (no value), con-lsta:FE08
- added E$51, E$60, E$63, E$72: (no value), con-lstb:MA04-1
- added E$52, E$64: (no value), con-wago-508:W237-4P
- added E$53, E$55, E$56, E$65, E$67, E$68: (no value), diode:DO34-7
- added E$54, E$66: (no value), con-wago-500:W237-102
- added E$57, E$69: (no value), con-lstb:MA03-2
- added E$58, E$59, E$70, E$71: (no value), con-lstb:MA06-1
Connections:
- new net S$33: E$50.3, E$51.4, E$52.4, E$60.4
- new net S$34: E$50.4, E$51.3, E$52.3, E$60.3
- new net S$57: E$50.5, E$51.2, E$52.2, E$60.2
- new net S$58: E$50.6, E$51.1, E$52.1, E$60.1
- new net S$61: E$49.8, E$53.C, E$58.1, E$59.1
- new net S$62: E$49.1, E$57.3, E$57.5, E$58.6, E$59.6
- new net S$63: E$53.A, E$57.1
- new net S$64: E$56.A, E$57.6
- new net S$65: E$55.A, E$57.4
- new net S$66: E$49.5, E$58.4, E$59.4
- new net S$67: E$49.6, E$58.3, E$59.3
- new net S$68: E$49.7, E$58.2, E$59.2
- new net S$69: E$49.2, E$58.5, E$59.5
- new net S$70: E$62.3, E$63.4, E$64.4, E$72.4
- new net S$71: E$62.4, E$63.3, E$64.3, E$72.3
- new net S$72: E$62.5, E$63.2, E$64.2, E$72.2
- new net S$73: E$62.6, E$63.1, E$64.1, E$72.1
- new net S$74: E$61.8, E$65.C, E$70.1, E$71.1
- new net S$75: E$61.1, E$69.3, E$69.5, E$70.6, E$71.6
- new net S$76: E$65.A, E$69.1
- new net S$77: E$68.A, E$69.6
- new net S$78: E$67.A, E$69.4
- new net S$79: E$61.5, E$70.4, E$71.4
- new net S$80: E$61.6, E$70.3, E$71.3
- new net S$81: E$61.7, E$70.2, E$71.2
- new net S$82: E$61.2, E$70.5, E$71.5
- net S$5: now also E$50.1, E$50.7, E$54.1, E$55.C, E$62.1, E$62.7, E$66.1, E$67.C
- net S$6: now also E$49.3, E$49.4, E$50.2, E$54.2, E$56.C, E$57.2, E$61.3, E$61.4, E$62.2, E$66.2, E$68.C, E$69.2
Routing:
- net S$6: track 222.8 -> 342.5 mm
- net S$5: track 179.2 -> 276.1 mm
- net S$74: track 0.00 -> 18.6 mm
- net S$61: track 0.00 -> 18.6 mm
- net S$57: track 0.00 -> 16.4 mm
- net S$34: track 0.00 -> 16.4 mm
- net S$72: track 0.00 -> 16.4 mm
- net S$71: track 0.00 -> 16.4 mm
- net S$70: track 0.00 -> 14.9 mm
- net S$58: track 0.00 -> 14.9 mm
- net S$33: track 0.00 -> 14.9 mm
- net S$73: track 0.00 -> 14.9 mm
- net S$62: track 0.00 -> 13.8 mm
- net S$75: track 0.00 -> 13.8 mm
- net S$65: track 0.00 -> 11.2 mm
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
Commit message: pcb
Parts:
- removed E$37, E$38, E$49, E$50, E$61, E$62: (no value), con-lsta:FE08
- removed E$39, E$48, E$51, E$60, E$63, E$72: (no value), con-lstb:MA04-1
- removed E$40, E$52, E$64: (no value), con-wago-508:W237-4P
- removed E$41, E$43, E$44, E$53, E$55, E$56, E$65, E$67, E$68: (no value), diode:DO34-7
- removed E$42, E$54, E$66: (no value), con-wago-500:W237-102
- removed E$45, E$57, E$69: (no value), con-lstb:MA03-2
- removed E$46, E$47, E$58, E$59, E$70, E$71: (no value), con-lstb:MA06-1
- added E$100, E$76, E$88: (no value), con-wago-508:W237-4P
- added E$101, E$103, E$104, E$77, E$79, E$80, E$89, E$91, E$92: (no value), diode:DO34-7
- added E$102, E$78, E$90: (no value), con-wago-500:W237-102
- added E$105, E$81, E$93: (no value), con-lstb:MA03-2
- added E$106, E$107, E$82, E$83, E$94, E$95: (no value), con-lstb:MA06-1
- added E$108, E$75, E$84, E$87, E$96, E$99: (no value), con-lstb:MA04-1
- added E$73, E$74, E$85, E$86, E$97, E$98: (no value), con-lsta:FE08
Connections:
- removed net S$33: E$50.3, E$51.4, E$52.4, E$60.4
- removed net S$34: E$50.4, E$51.3, E$52.3, E$60.3
- removed net S$44: E$38.3, E$39.4, E$40.4, E$48.4
- removed net S$45: E$38.4, E$39.3, E$40.3, E$48.3
- removed net S$46: E$38.5, E$39.2, E$40.2, E$48.2
- removed net S$47: E$38.6, E$39.1, E$40.1, E$48.1
- removed net S$48: E$37.8, E$41.C, E$46.1, E$47.1
- removed net S$49: E$37.1, E$45.3, E$45.5, E$46.6, E$47.6
- removed net S$5: E$14.1, E$14.7, E$18.1, E$19.C, E$2.1, E$2.7, E$26.1, E$26.7, E$30.1, E$31.C, E$38.1, E$38.7, E$42.1, E$43.C, E$50.1, E$50.7, E$54.1, E$55.C, E$62.1, E$62.7, E$66.1, E$67.C, E$7.1, E$9.C
- removed net S$50: E$41.A, E$45.1
- removed net S$51: E$44.A, E$45.6
- removed net S$52: E$43.A, E$45.4
- removed net S$53: E$37.5, E$46.4, E$47.4
- removed net S$54: E$37.6, E$46.3, E$47.3
- removed net S$55: E$37.7, E$46.2, E$47.2
- removed net S$56: E$37.2, E$46.5, E$47.5
- removed net S$57: E$50.5, E$51.2, E$52.2, E$60.2
- removed net S$58: E$50.6, E$51.1, E$52.1, E$60.1
- removed net S$61: E$49.8, E$53.C, E$58.1, E$59.1
- removed net S$62: E$49.1, E$57.3, E$57.5, E$58.6, E$59.6
- removed net S$63: E$53.A, E$57.1
- removed net S$64: E$56.A, E$57.6
- removed net S$65: E$55.A, E$57.4
- removed net S$66: E$49.5, E$58.4, E$59.4
- removed net S$67: E$49.6, E$58.3, E$59.3
- removed net S$68: E$49.7, E$58.2, E$59.2
- removed net S$69: E$49.2, E$58.5, E$59.5
- removed net S$70: E$62.3, E$63.4, E$64.4, E$72.4
- removed net S$71: E$62.4, E$63.3, E$64.3, E$72.3
- removed net S$72: E$62.5, E$63.2, E$64.2, E$72.2
- removed net S$73: E$62.6, E$63.1, E$64.1, E$72.1
- removed net S$74: E$61.8, E$65.C, E$70.1, E$71.1
- removed net S$75: E$61.1, E$69.3, E$69.5, E$70.6, E$71.6
- removed net S$76: E$65.A, E$69.1
- removed net S$77: E$68.A, E$69.6
- removed net S$78: E$67.A, E$69.4
- removed net S$79: E$61.5, E$70.4, E$71.4
- removed net S$80: E$61.6, E$70.3, E$71.3
- removed net S$81: E$61.7, E$70.2, E$71.2
- removed net S$82: E$61.2, E$70.5, E$71.5
- new net S$100: E$86.5, E$87.2, E$88.2, E$96.2
- new net S$101: E$86.6, E$87.1, E$88.1, E$96.1
- new net S$102: E$85.8, E$89.C, E$94.1, E$95.1
- new net S$103: E$85.1, E$93.3, E$93.5, E$94.6, E$95.6
- new net S$104: E$89.A, E$93.1
- new net S$105: E$92.A, E$93.6
- new net S$106: E$91.A, E$93.4
- new net S$107: E$85.5, E$94.4, E$95.4
- new net S$108: E$85.6, E$94.3, E$95.3
- new net S$109: E$85.7, E$94.2, E$95.2
- new net S$110: E$85.2, E$94.5, E$95.5
- new net S$111: E$100.4, E$108.4, E$98.3, E$99.4
- new net S$112: E$100.3, E$108.3, E$98.4, E$99.3
- new net S$113: E$100.2, E$108.2, E$98.5, E$99.2
- new net S$114: E$100.1, E$108.1, E$98.6, E$99.1
- new net S$115: E$101.C, E$106.1, E$107.1, E$97.8
- new net S$116: E$105.3, E$105.5, E$106.6, E$107.6, E$97.1
- new net S$117: E$101.A, E$105.1
- new net S$118: E$104.A, E$105.6
- new net S$119: E$103.A, E$105.4
- new net S$120: E$106.4, E$107.4, E$97.5
- new net S$121: E$106.3, E$107.3, E$97.6
- new net S$122: E$106.2, E$107.2, E$97.7
- new net S$123: E$106.5, E$107.5, E$97.2
- new net S$60: E$14.1, E$14.7, E$18.1, E$19.C, E$2.1, E$2.7, E$26.1, E$26.7, E$30.1, E$31.C, E$7.1, E$9.C
- new net S$83: E$102.1, E$103.C, E$74.1, E$74.7, E$78.1, E$79.C, E$86.1, E$86.7, E$90.1, E$91.C, E$98.1, E$98.7
- new net S$84: E$102.2, E$104.C, E$105.2, E$73.3, E$73.4, E$74.2, E$78.2, E$80.C, E$81.2, E$85.3, E$85.4, E$86.2, E$90.2, E$92.C, E$93.2, E$97.3, E$97.4, E$98.2
- new net S$85: E$74.3, E$75.4, E$76.4, E$84.4
- new net S$86: E$74.4, E$75.3, E$76.3, E$84.3
- new net S$87: E$74.5, E$75.2, E$76.2, E$84.2
- new net S$88: E$74.6, E$75.1, E$76.1, E$84.1
- new net S$89: E$73.8, E$77.C, E$82.1, E$83.1
- new net S$90: E$73.1, E$81.3, E$81.5, E$82.6, E$83.6
- new net S$91: E$77.A, E$81.1
- new net S$92: E$80.A, E$81.6
- new net S$93: E$79.A, E$81.4
- new net S$94: E$73.5, E$82.4, E$83.4
- new net S$95: E$73.6, E$82.3, E$83.3
- new net S$96: E$73.7, E$82.2, E$83.2
- new net S$97: E$73.2, E$82.5, E$83.5
- new net S$98: E$86.3, E$87.4, E$88.4, E$96.4
- new net S$99: E$86.4, E$87.3, E$88.3, E$96.3
- net S$6: no longer E$37.3, E$37.4, E$38.2, E$42.2, E$44.C, E$45.2, E$49.3, E$49.4, E$50.2, E$54.2, E$56.C, E$57.2, E$61.3, E$61.4, E$62.2, E$66.2, E$68.C, E$69.2
Routing:
- net S$5: track 276.1 -> 0.00 mm
- net S$6: track 342.5 -> 163.0 mm
- net S$84: track 0.00 -> 163.0 mm
- net S$83: track 0.00 -> 132.0 mm
- net S$60: track 0.00 -> 131.2 mm
- net S$74: track 18.6 -> 0.00 mm
- net S$89: track 0.00 -> 18.6 mm
- net S$102: track 0.00 -> 18.6 mm
- net S$61: track 18.6 -> 0.00 mm
- net S$48: track 18.6 -> 0.00 mm
- net S$115: track 0.00 -> 18.6 mm
- net S$57: track 16.4 -> 0.00 mm
- net S$34: track 16.4 -> 0.00 mm
- net S$72: track 16.4 -> 0.00 mm
- net S$71: track 16.4 -> 0.00 mm
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
Commit message: pcb
Parts:
- added E$40, E$41, E$42: (no value), con-molex:70543-22
- moved E$100 12.7 mm to (116.8, 74.9)
- moved E$101 12.7 mm to (94.0, 72.4)
- moved E$102 12.7 mm to (105.4, 58.4)
- moved E$103 12.7 mm to (101.6, 63.7)
- moved E$105 12.7 mm to (91.4, 62.2)
- moved E$106 12.7 mm to (85.1, 74.9)
- moved E$107 12.7 mm to (82.5, 74.9)
- moved E$108 12.7 mm to (109.2, 74.9)
- moved E$73 12.7 mm to (90.2, 16.5)
- moved E$74 12.7 mm to (102.9, 16.5)
- moved E$75 12.7 mm to (106.7, 16.5)
- moved E$76 12.7 mm to (116.8, 16.5)
- moved E$77 12.7 mm to (94.0, 14.0)
- moved E$78 12.7 mm to (105.4, 0.00)
- moved E$79 12.7 mm to (101.6, 5.32)
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Connections:
- new net S$33: E$40.2, E$41.2
- new net S$34: E$40.3, E$41.3
- new net S$44: E$40.5, E$41.5
- new net S$45: E$40.22, E$41.4
- new net S$5: E$40.1, E$41.1
- net S$12: now also E$40.8
- net S$13: now also E$40.9
- net S$14: now also E$40.10
- net S$15: now also E$40.7
- net S$22: now also E$40.17
- net S$23: now also E$40.12
- net S$27: now also E$40.14
- net S$28: now also E$40.15
- net S$29: now also E$40.16
- net S$30: now also E$40.13
- net S$35: now also E$41.7
- net S$36: now also E$40.18
- net S$40: now also E$40.20
- net S$41: now also E$40.21
- net S$42: now also E$41.6
- net S$43: now also E$40.19
- net S$7: now also E$40.11
- net S$8: now also E$40.6
Routing:
- net S$45: track 0.00 -> 55.9 mm
- net S$23: track 13.8 -> 39.7 mm
- net S$30: track 8.67 -> 33.9 mm
- net S$27: track 8.67 -> 33.1 mm
- net S$28: track 8.67 -> 32.4 mm
- net S$29: track 8.67 -> 31.6 mm
- net S$22: track 18.6 -> 40.8 mm
- net S$5: track 0.00 -> 12.7 mm
- net S$44: track 0.00 -> 12.7 mm
- net S$34: track 0.00 -> 12.7 mm
- net S$33: track 0.00 -> 12.7 mm
- net S$8: track 13.8 -> 26.5 mm
- net S$7: track 18.6 -> 31.3 mm
- net S$13: track 8.67 -> 21.4 mm
- net S$15: track 8.67 -> 21.4 mm
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