File: Grbl_Esp32/src/custom/pcb/grbl_shift_register.brd (EAGLE design)
At the start: 75 parts

Commit message: pcb
Parts:
- moved E$40 2.54 mm to (53.3, 67.3)
- moved E$41 2.54 mm to (66.0, 67.3)
Connections:
- net S$115: now also E$41.8
- net S$116: now also E$41.13
- net S$120: now also E$41.11
- net S$121: now also E$41.10
- net S$122: now also E$41.9
- net S$123: now also E$41.12
Routing:
- net S$35: track 18.6 -> 105.5 mm
- net S$42: track 8.67 -> 94.8 mm
- net S$41: track 8.67 -> 45.9 mm
- net S$40: track 8.67 -> 45.2 mm
- net S$43: track 8.67 -> 44.4 mm
- net S$36: track 13.8 -> 48.7 mm
- net S$23: track 39.7 -> 34.8 mm
- net S$30: track 33.9 -> 30.4 mm
- net S$27: track 33.1 -> 30.4 mm
- net S$8: track 26.5 -> 29.0 mm
- net S$7: track 31.3 -> 33.9 mm
- net S$15: track 21.4 -> 23.9 mm
- net S$14: track 21.4 -> 23.9 mm
- net S$13: track 21.4 -> 23.9 mm
- net S$12: track 21.4 -> 23.9 mm
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
Commit message: pcb
Connections:
- net S$102: now also E$41.14
- net S$103: now also E$41.19
- net S$107: now also E$41.17
- net S$108: now also E$41.16
- net S$109: now also E$41.15
- net S$110: now also E$41.18
Routing:
- net S$102: track 18.6 -> 40.3 mm
- net S$109: track 8.67 -> 29.6 mm
- net S$110: track 8.67 -> 28.9 mm
- net S$108: track 8.67 -> 28.9 mm
- net S$107: track 8.67 -> 28.9 mm
- net S$103: track 13.8 -> 33.9 mm
- net S$123: track 8.67 -> 27.3 mm
- net S$122: track 8.67 -> 27.3 mm
- net S$121: track 8.67 -> 27.3 mm
- net S$120: track 8.67 -> 27.3 mm
- net S$116: track 13.8 -> 32.4 mm
- net S$115: track 18.6 -> 37.2 mm
- net S$45: track 55.9 -> 59.8 mm
Changed lines of the file:
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@@
 <wire x1="86.36" y1="52.07" x2="85.09" y2="52.07" width="0.8128" layer="16"/>
 <wire x1="85.09" y1="52.07" x2="82.55" y2="52.07" width="0.8128" layer="16"/>
+<contactref element="E$41" pad="14"/>
+<wire x1="66.04" y1="60.96" x2="69.85" y2="60.96" width="0.8128" layer="16"/>
+<wire x1="69.85" y1="60.96" x2="74.93" y2="55.88" width="0.8128" layer="16"/>
+<wire x1="74.93" y1="53.34" x2="76.2" y2="52.07" width="0.8128" layer="16"/>
+<wire x1="76.2" y1="52.07" x2="82.55" y2="52.07" width="0.8128" layer="16"/>
+<wire x1="74.93" y1="55.88" x2="74.93" y2="53.34" width="0.8128" layer="16"/>
 </signal>
 <signal name="S$103">
@@
 <wire x1="88.9" y1="36.83" x2="86.36" y2="39.37" width="0.8128" layer="16"/>
 <wire x1="85.09" y1="39.37" x2="82.55" y2="39.37" width="0.8128" layer="16"/>
+<contactref element="E$41" pad="19"/>
+<wire x1="66.04" y1="48.26" x2="67.31" y2="48.26" width="0.8128" layer="16"/>
+<wire x1="67.31" y1="48.26" x2="76.2" y2="39.37" width="0.8128" layer="16"/>
+<wire x1="76.2" y1="39.37" x2="82.55" y2="39.37" width="0.8128" layer="16"/>
 </signal>
 <signal name="S$104">
@@
 <wire x1="88.9" y1="46.99" x2="86.36" y2="44.45" width="0.8128" layer="16"/>
 <wire x1="85.09" y1="44.45" x2="82.55" y2="44.45" width="0.8128" layer="16"/>
+<contactref element="E$41" pad="17"/>
+<wire x1="66.04" y1="53.34" x2="67.31" y2="53.34" width="0.8128" layer="16"/>
+<wire x1="67.31" y1="53.34" x2="76.2" y2="44.45" width="0.8128" layer="16"/>
+<wire x1="76.2" y1="44.45" x2="82.55" y2="44.45" width="0.8128" layer="16"/>
 </signal>
 <signal name="S$108">
@@
 <wire x1="86.36" y1="46.99" x2="85.09" y2="46.99" width="0.8128" layer="16"/>
 <wire x1="85.09" y1="46.99" x2="82.55" y2="46.99" width="0.8128" layer="16"/>
+<contactref element="E$41" pad="16"/>
+<wire x1="66.04" y1="55.88" x2="67.31" y2="55.88" width="0.8128" layer="16"/>
+<wire x1="76.2" y1="46.99" x2="82.55" y2="46.99" width="0.8128" layer="16"/>
+<wire x1="67.31" y1="55.88" x2="76.2" y2="46.99" width="0.8128" layer="16"/>
 </signal>
 <signal name="S$109">
@@
 <wire x1="86.36" y1="49.53" x2="85.09" y2="49.53" width="0.8128" layer="16"/>
 <wire x1="85.09" y1="49.53" x2="82.55" y2="49.53" width="0.8128" layer="16"/>
+<contactref element="E$41" pad="15"/>
+<wire x1="66.04" y1="58.42" x2="68.58" y2="58.42" width="0.8128" layer="16"/>
+<wire x1="68.58" y1="58.42" x2="72.39" y2="54.61" width="0.8128" layer="16"/>
+<wire x1="72.39" y1="54.61" x2="72.39" y2="53.34" width="0.8128" layer="16"/>
+<wire x1="72.39" y1="53.34" x2="76.2" y2="49.53" width="0.8128" layer="16"/>
+<wire x1="76.2" y1="49.53" x2="82.55" y2="49.53" width="0.8128" layer="16"/>
 </signal>
 <signal name="S$110">
@@
 <wire x1="86.36" y1="41.91" x2="85.09" y2="41.91" width="0.8128" layer="16"/>
 <wire x1="85.09" y1="41.91" x2="82.55" y2="41.91" width="0.8128" layer="16"/>
+<contactref element="E$41" pad="18"/>
+<wire x1="66.04" y1="50.8" x2="67.31" y2="50.8" width="0.8128" layer="16"/>
+<wire x1="76.2" y1="41.91" x2="82.55" y2="41.91" width="0.8128" layer="16"/>
+<wire x1="67.31" y1="50.8" x2="76.2" y2="41.91" width="0.8128" layer="16"/>
 </signal>
 <signal name="S$111">
@@
 <wire x1="85.09" y1="81.28" x2="82.55" y2="81.28" width="0.8128" layer="16"/>
 <contactref element="E$41" pad="8"/>
-<wire x1="66.04" y1="76.2" x2="82.55" y2="81.28" width="0" layer="19" extent="1-16"/>
+<wire x1="66.04" y1="76.2" x2="68.58" y2="76.2" width="0.8128" layer="16"/>
+<wire x1="68.58" y1="76.2" x2="73.66" y2="81.28" width="0.8128" layer="16"/>
+<wire x1="73.66" y1="81.28" x2="82.55" y2="81.28" width="0.8128" layer="16"/>
 </signal>
 <signal name="S$116">
@@
 <wire x1="85.09" y1="68.58" x2="82.55" y2="68.58" width="0.8128" layer="16"/>
 <contactref element="E$41" pad="13"/>
-<wire x1="66.04" y1="63.5" x2="82.55" y2="68.58" width="0" layer="19" extent="1-16"/>
+<wire x1="66.04" y1="63.5" x2="68.58" y2="63.5" width="0.8128" layer="16"/>
+<wire x1="68.58" y1="63.5" x2="73.66" y2="68.58" width="0.8128" layer="16"/>
+<wire x1="73.66" y1="68.58" x2="82.55" y2="68.58" width="0.8128" layer="16"/>
 </signal>
 <signal name="S$117">
@@
 <wire x1="85.09" y1="73.66" x2="82.55" y2="73.66" width="0.8128" layer="16"/>
 <contactref element="E$41" pad="11"/>
-<wire x1="66.04" y1="68.58" x2="82.55" y2="73.66" width="0" layer="19" extent="1-16"/>
+<wire x1="66.04" y1="68.58" x2="68.58" y2="68.58" width="0.8128" layer="16"/>
+<wire x1="68.58" y1="68.58" x2="73.66" y2="73.66" width="0.8128" layer="16"/>
+<wire x1="73.66" y1="73.66" x2="82.55" y2="73.66" width="0.8128" layer="16"/>
 </signal>
 <signal name="S$121">
@@
 <wire x1="85.09" y1="76.2" x2="82.55" y2="76.2" width="0.8128" layer="16"/>
 <contactref element="E$41" pad="10"/>
-<wire x1="66.04" y1="71.12" x2="82.55" y2="76.2" width="0" layer="19" extent="1-16"/>
+<wire x1="66.04" y1="71.12" x2="68.58" y2="71.12" width="0.8128" layer="16"/>
+<wire x1="68.58" y1="71.12" x2="73.66" y2="76.2" width="0.8128" layer="16"/>
+<wire x1="73.66" y1="76.2" x2="82.55" y2="76.2" width="0.8128" layer="16"/>
 </signal>
 <signal name="S$122">
@@
 <wire x1="85.09" y1="78.74" x2="82.55" y2="78.74" width="0.8128" layer="16"/>
 <contactref element="E$41" pad="9"/>
-<wire x1="66.04" y1="73.66" x2="82.55" y2="78.74" width="0" layer="19" extent="1-16"/>
+<wire x1="66.04" y1="73.66" x2="68.58" y2="73.66" width="0.8128" layer="16"/>
+<wire x1="68.58" y1="73.66" x2="73.66" y2="78.74" width="0.8128" layer="16"/>
+<wire x1="73.66" y1="78.74" x2="82.55" y2="78.74" width="0.8128" layer="16"/>
 </signal>
 <signal name="S$123">
@@
 <wire x1="85.09" y1="71.12" x2="82.55" y2="71.12" width="0.8128" layer="16"/>
 <contactref element="E$41" pad="12"/>
-<wire x1="66.04" y1="66.04" x2="82.55" y2="71.12" width="0" layer="19" extent="1-16"/>
+<wire x1="66.04" y1="66.04" x2="68.58" y2="66.04" width="0.8128" layer="16"/>
+<wire x1="73.66" y1="71.12" x2="82.55" y2="71.12" width="0.8128" layer="16"/>
+<wire x1="68.58" y1="66.04" x2="73.66" y2="71.12" width="0.8128" layer="16"/>
 </signal>
 <signal name="S$5">
@@
 <contactref element="E$41" pad="4"/>
 <wire x1="55.88" y1="40.64" x2="53.34" y2="40.64" width="0.8128" layer="16"/>
-<wire x1="64.68010625" y1="82.55" x2="60.96" y2="82.55" width="0.8128" layer="16"/>
+<wire x1="60.96" y1="82.55" x2="64.68010625" y2="82.55" width="0.8128" layer="16"/>
 <wire x1="67.31" y1="86.36" x2="66.04" y2="86.36" width="0.8128" layer="16"/>
 <wire x1="68.58" y1="85.09" x2="67.31" y2="86.36" width="0.8128" layer="16"/>
-<wire x1="68.58" y1="85.09" x2="68.58" y2="82.55" width="0.8128" layer="16"/>
+<wire x1="68.58" y1="82.55" x2="68.58" y2="85.09" width="0.8128" layer="16"/>
 <wire x1="57.15" y1="41.91" x2="55.88" y2="40.64" width="0.8128" layer="16"/>
 <wire x1="60.96" y1="82.55" x2="57.15" y2="78.74" width="0.8128" layer="16"/>
 <wire x1="57.15" y1="78.74" x2="57.15" y2="41.91" width="0.8128" layer="16"/>
-<wire x1="64.68010625" y1="82.55" x2="68.58" y2="82.55" width="0" layer="19" extent="16-16"/>
+<wire x1="64.68010625" y1="82.55" x2="68.58" y2="82.55" width="0.6096" layer="16"/>
 </signal>
 </signals>

Commit message: pcb
Parts:
- moved E$75 5.08 mm to (101.6, 16.5)
- moved E$87 5.08 mm to (101.6, 45.7)
- moved E$99 5.08 mm to (101.6, 74.9)
- moved E$100 5.08 mm to (111.8, 74.9)
- moved E$101 5.08 mm to (88.9, 72.4)
- moved E$102 5.08 mm to (100.3, 58.4)
- moved E$103 5.08 mm to (96.5, 63.7)
- moved E$104 5.08 mm to (87.6, 58.4)
- moved E$105 5.08 mm to (86.4, 62.2)
- moved E$106 5.08 mm to (80.0, 74.9)
- moved E$107 5.08 mm to (77.5, 74.9)
- moved E$108 5.08 mm to (104.1, 74.9)
- moved E$73 5.08 mm to (85.1, 16.5)
- moved E$74 5.08 mm to (97.8, 16.5)
- moved E$76 5.08 mm to (111.8, 16.5)
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Connections:
- removed net S$83: E$102.1, E$103.C, E$74.1, E$74.7, E$78.1, E$79.C, E$86.1, E$86.7, E$90.1, E$91.C, E$98.1, E$98.7
- removed net S$84: E$102.2, E$104.C, E$105.2, E$73.3, E$73.4, E$74.2, E$78.2, E$80.C, E$81.2, E$85.3, E$85.4, E$86.2, E$90.2, E$92.C, E$93.2, E$97.3, E$97.4, E$98.2
- net S$6: now also E$102.2, E$104.C, E$105.2, E$73.3, E$73.4, E$74.2, E$78.2, E$80.C, E$81.2, E$85.3, E$85.4, E$86.2, E$90.2, E$92.C, E$93.2, E$97.3, E$97.4, E$98.2
- net S$60: now also E$102.1, E$103.C, E$74.1, E$74.7, E$78.1, E$79.C, E$86.1, E$86.7, E$90.1, E$91.C, E$98.1, E$98.7
Routing:
- net S$6: track 163.0 -> 412.0 mm
- net S$60: track 131.2 -> 355.1 mm
- net S$84: track 163.0 -> 0.00 mm
- net S$83: track 132.0 -> 0.00 mm
- net S$115: track 37.2 -> 32.1 mm
- net S$102: track 40.3 -> 35.2 mm
- net S$123: track 27.3 -> 22.2 mm
- net S$122: track 27.3 -> 22.2 mm
- net S$121: track 27.3 -> 22.2 mm
- net S$120: track 27.3 -> 22.2 mm
- net S$110: track 28.9 -> 23.8 mm
- net S$108: track 28.9 -> 23.8 mm
- net S$109: track 29.6 -> 24.5 mm
- net S$107: track 28.9 -> 23.8 mm
- net S$116: track 32.4 -> 27.3 mm
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
Commit message: pcb
Parts:
- moved E$42 167.0 mm to (62.2, -16.5)
- moved E$101 6.35 mm to (83.8, 76.2)
- moved E$86 6.35 mm to (92.7, 49.5)
- moved E$89 6.35 mm to (83.8, 47.0)
- moved E$77 6.35 mm to (83.8, 17.8)
- moved E$74 6.35 mm to (92.7, 20.3)
- moved E$105 6.35 mm to (81.3, 66.0)
- moved E$98 6.35 mm to (92.7, 78.7)
- moved E$85 6.35 mm to (80.0, 49.5)
- moved E$87 6.35 mm to (96.5, 49.5)
- moved E$88 6.35 mm to (106.7, 49.5)
- moved E$90 6.35 mm to (95.2, 33.0)
- moved E$91 6.35 mm to (91.4, 38.3)
- moved E$92 6.35 mm to (82.5, 33.0)
- moved E$94 6.35 mm to (74.9, 49.5)
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Connections:
- net S$121 renamed S$47
- net S$122 renamed S$46
Routing:
- net S$60: track 355.1 -> 347.3 mm
- net S$6: track 412.0 -> 419.5 mm
- net S$103: track 28.9 -> 23.5 mm
- net S$109: track 24.5 -> 19.7 mm
- net S$110: track 23.8 -> 19.7 mm
- net S$102: track 35.2 -> 31.1 mm
- net S$107: track 23.8 -> 19.7 mm
- net S$108: track 23.8 -> 19.7 mm
- net S$5: track 12.7 -> 10.2 mm
- net S$44: track 12.7 -> 10.2 mm
- net S$42: track 94.8 -> 92.2 mm
- net S$34: track 12.7 -> 10.2 mm
- net S$33: track 12.7 -> 10.2 mm
- net S$35: track 105.5 -> 102.9 mm
- net S$116: track 27.3 -> 25.8 mm
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