File: Grbl_Esp32/src/custom/pcb/grbl_shift_register.brd (EAGLE design)
At the start: 75 parts

Commit message: pcb
Parts:
- removed E$100, E$16, E$28, E$5, E$76, E$88: (no value), con-wago-508:W237-4P
Connections:
- net S$1: no longer E$5.4
- net S$100: no longer E$88.2
- net S$101: no longer E$88.1
- net S$111: no longer E$100.4
- net S$112: no longer E$100.3
- net S$113: no longer E$100.2
- net S$114: no longer E$100.1
- net S$16: no longer E$16.4
- net S$17: no longer E$16.3
- net S$18: no longer E$16.2
- net S$19: no longer E$16.1
- net S$2: no longer E$5.3
- net S$20: no longer E$28.4
- net S$21: no longer E$28.3
- net S$3: no longer E$5.2
- net S$31: no longer E$28.2
- net S$32: no longer E$28.1
- net S$4: no longer E$5.1
- net S$85: no longer E$76.4
- net S$86: no longer E$76.3
- net S$87: no longer E$76.2
- net S$88: no longer E$76.1
- net S$98: no longer E$88.4
- net S$99: no longer E$88.3
Routing:
- net S$99: track 16.4 -> 6.35 mm
- net S$87: track 16.4 -> 6.35 mm
- net S$86: track 16.4 -> 6.35 mm
- net S$18: track 16.4 -> 6.35 mm
- net S$113: track 16.4 -> 6.35 mm
- net S$31: track 16.4 -> 6.35 mm
- net S$3: track 16.4 -> 6.35 mm
- net S$21: track 16.4 -> 6.35 mm
- net S$2: track 16.4 -> 6.35 mm
- net S$17: track 16.4 -> 6.35 mm
- net S$4: track 14.9 -> 6.35 mm
- net S$16: track 14.9 -> 6.35 mm
- net S$1: track 14.9 -> 6.35 mm
- net S$98: track 14.9 -> 6.35 mm
- net S$88: track 14.9 -> 6.35 mm
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
Commit message: pcb
Routing:
- net S$89: track 17.3 -> 18.6 mm
- net S$115: track 30.7 -> 32.0 mm
Changed lines of the file:
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@@
 <contactref element="E$77" pad="C"/>
 <contactref element="E$73" pad="8"/>
-<wire x1="83.82" y1="26.67" x2="81.28" y2="29.21" width="0.8128" layer="16"/>
+<wire x1="81.28" y1="29.21" x2="83.82" y2="26.67" width="0.8128" layer="16"/>
 <wire x1="83.82" y1="26.67" x2="83.82" y2="21.59" width="0.8128" layer="16"/>
 <contactref element="E$82" pad="1"/>
@@
 <wire x1="76.2" y1="26.67" x2="74.93" y2="26.67" width="0.8128" layer="16"/>
 <wire x1="74.93" y1="26.67" x2="72.39" y2="26.67" width="0.8128" layer="16"/>
+<wire x1="80.01" y1="29.21" x2="81.28" y2="29.21" width="0.8128" layer="16"/>
 </signal>
 <signal name="S$90">
@@
 <contactref element="E$101" pad="C"/>
 <contactref element="E$97" pad="8"/>
-<wire x1="83.82" y1="85.09" x2="81.28" y2="87.63" width="0.8128" layer="16"/>
+<wire x1="81.28" y1="87.63" x2="83.82" y2="85.09" width="0.8128" layer="16"/>
 <wire x1="83.82" y1="85.09" x2="83.82" y2="80.01" width="0.8128" layer="16"/>
 <contactref element="E$106" pad="1"/>
@@
 <wire x1="63.5" y1="76.2" x2="63.58989375" y2="76.2" width="0.8128" layer="16"/>
 <wire x1="66.04" y1="78.65010625" x2="66.04" y2="80.01" width="0.6096" layer="16"/>
-<wire x1="80.01" y1="87.63" x2="81.28" y2="87.63" width="0" layer="19" extent="16-16"/>
+<wire x1="80.01" y1="87.63" x2="81.28" y2="87.63" width="0.8128" layer="16"/>
 </signal>
 <signal name="S$116">

Commit message: pcb
Parts:
- added E$16, E$5: (no value), con-lstb:MA05-1
- added E$28, E$37, E$39: (no value), diode:DO34-7
- added E$38, E$43: (no value), con-molex:22-23-2021
- added E$44, E$45, E$46, E$47, E$48, E$49: (no value), con-wago-500:W237-102
- moved E$42 9.16 mm to (57.1, -8.89), flipped to the bottom, turned to 180 degrees
Connections:
- new net S$48: E$16.2, E$40.4, E$5.2
- net S$33: now also E$16.4, E$5.4
- net S$34: now also E$16.3, E$5.3
- net S$44: now also E$28.A, E$38.2; no longer E$40.5, E$41.5
- net S$5: now also E$16.5, E$38.1, E$5.5
- net S$6: now also E$16.1, E$28.C, E$40.5, E$41.5, E$5.1
Routing:
- net S$6: track 419.5 -> 469.3 mm
- net S$5: track 10.2 -> 22.9 mm
- net S$48: track 0.00 -> 7.62 mm
- net S$34: track 10.2 -> 17.8 mm
- net S$33: track 10.2 -> 17.8 mm
- net S$44: track 10.2 -> 3.07 mm
- net S$60: track 347.3 -> 346.6 mm

Commit message: pcb
Connections:
- new net S$49: E$14.8, E$2.8, E$26.8, E$44.2, E$45.1, E$46.1, E$47.1, E$48.1, E$49.1, E$74.8, E$86.8, E$98.8
- net S$60: now also E$44.1, E$45.2, E$46.2, E$47.2, E$48.2, E$49.2
Routing:
- net S$49: track 0.00 -> 218.5 mm
- net S$60: track 346.6 -> 392.4 mm
Changed lines of the file:
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@@
 <wire x1="97.75" y1="34.29" x2="94.575" y2="31.115" width="0.8128" layer="16"/>
 <wire x1="94.575" y1="31.115" x2="90.805" y2="31.115" width="0.8128" layer="16"/>
+<contactref element="E$48" pad="2"/>
+<contactref element="E$47" pad="2"/>
+<contactref element="E$49" pad="2"/>
+<contactref element="E$46" pad="2"/>
+<contactref element="E$45" pad="2"/>
+<contactref element="E$44" pad="1"/>
+<wire x1="10.16" y1="68.54" x2="10.2" y2="68.58" width="0.8128" layer="16"/>
+<wire x1="10.2" y1="68.58" x2="17.78" y2="68.58" width="0.8128" layer="16"/>
+<wire x1="10.16" y1="39.33" x2="10.2" y2="39.37" width="0.8128" layer="16"/>
+<wire x1="10.2" y1="39.37" x2="17.78" y2="39.37" width="0.8128" layer="16"/>
+<wire x1="17.78" y1="10.16" x2="17.74" y2="10.12" width="0.8128" layer="16"/>
+<wire x1="17.74" y1="10.12" x2="10.16" y2="10.12" width="0.8128" layer="16"/>
+<wire x1="100.33" y1="26.71" x2="100.29" y2="26.67" width="0.8128" layer="16"/>
+<wire x1="100.29" y1="26.67" x2="92.71" y2="26.67" width="0.8128" layer="16"/>
+<wire x1="100.33" y1="55.92" x2="100.29" y2="55.88" width="0.8128" layer="16"/>
+<wire x1="100.29" y1="55.88" x2="92.71" y2="55.88" width="0.8128" layer="16"/>
+<wire x1="100.33" y1="85.13" x2="100.29" y2="85.09" width="0.8128" layer="16"/>
+<wire x1="100.29" y1="85.09" x2="92.71" y2="85.09" width="0.8128" layer="16"/>
 </signal>
 <signal name="S$6">
@@
 <wire x1="36.83" y1="92.71" x2="38.1" y2="93.98" width="0.8128" layer="16"/>
 </signal>
+<signal name="S$49">
+<contactref element="E$44" pad="2"/>
+<contactref element="E$98" pad="8"/>
+<contactref element="E$86" pad="8"/>
+<contactref element="E$45" pad="1"/>
+<contactref element="E$74" pad="8"/>
+<contactref element="E$46" pad="1"/>
+<contactref element="E$26" pad="8"/>
+<contactref element="E$49" pad="1"/>
+<contactref element="E$14" pad="8"/>
+<contactref element="E$47" pad="1"/>
+<contactref element="E$2" pad="8"/>
+<contactref element="E$48" pad="1"/>
+<wire x1="92.71" y1="87.63" x2="96.52" y2="87.63" width="0.8128" layer="16"/>
+<wire x1="99.06" y1="90.17" x2="100.29" y2="90.17" width="0.8128" layer="16"/>
+<wire x1="100.29" y1="90.17" x2="100.33" y2="90.13" width="0.8128" layer="16"/>
+<wire x1="96.52" y1="87.63" x2="99.06" y2="90.17" width="0.8128" layer="16"/>
+<wire x1="100.33" y1="90.13" x2="101.56" y2="90.13" width="0.8128" layer="16"/>
+<wire x1="101.56" y1="90.13" x2="101.6" y2="90.17" width="0.8128" layer="16"/>
+<wire x1="101.6" y1="90.17" x2="102.87" y2="88.9" width="0.8128" layer="16"/>
+<wire x1="102.87" y1="88.9" x2="102.87" y2="83.82" width="0.8128" layer="16"/>
+<wire x1="102.87" y1="83.82" x2="101.6" y2="82.55" width="0.8128" layer="16"/>
+<wire x1="101.6" y1="82.55" x2="101.6" y2="73.66" width="0.8128" layer="16"/>
+<wire x1="100.33" y1="60.92" x2="97.83" y2="58.42" width="0.8128" layer="16"/>
+<wire x1="97.83" y1="58.42" x2="92.71" y2="58.42" width="0.8128" layer="16"/>
+<wire x1="100.33" y1="60.92" x2="101.56" y2="60.92" width="0.8128" layer="16"/>
+<wire x1="101.56" y1="60.92" x2="101.6" y2="60.96" width="0.8128" layer="16"/>
+<wire x1="101.6" y1="60.96" x2="102.87" y2="59.69" width="0.8128" layer="16"/>
+<wire x1="102.87" y1="54.61" x2="101.6" y2="53.34" width="0.8128" layer="16"/>
+<wire x1="101.6" y1="53.34" x2="101.6" y2="44.45" width="0.8128" layer="16"/>
+<wire x1="101.6" y1="44.45" x2="100.33" y2="43.18" width="0.8128" layer="16"/>
+<wire x1="100.33" y1="43.18" x2="100.33" y2="31.71" width="0.8128" layer="16"/>
+<wire x1="102.87" y1="59.69" x2="102.87" y2="54.61" width="0.8128" layer="16"/>
+<wire x1="101.6" y1="73.66" x2="100.33" y2="72.39" width="0.8128" layer="16"/>
+<wire x1="100.33" y1="72.39" x2="100.33" y2="60.92" width="0.8128" layer="16"/>
+<wire x1="97.83" y1="29.21" x2="100.33" y2="31.71" width="0.8128" layer="16"/>
+<wire x1="92.71" y1="29.21" x2="97.83" y2="29.21" width="0.8128" layer="16"/>
+<wire x1="100.33" y1="31.71" x2="101.56" y2="31.71" width="0.8128" layer="16"/>
+<wire x1="101.56" y1="31.71" x2="101.6" y2="31.75" width="0.8128" layer="16"/>
+<wire x1="101.6" y1="31.75" x2="102.87" y2="30.48" width="0.8128" layer="16"/>
+<wire x1="102.87" y1="25.4" x2="101.6" y2="24.13" width="0.8128" layer="16"/>
+<wire x1="101.6" y1="24.13" x2="101.6" y2="13.97" width="0.8128" layer="16"/>
+<wire x1="101.6" y1="13.97" x2="100.33" y2="12.7" width="0.8128" layer="16"/>
+<wire x1="100.33" y1="1.27" x2="99.06" y2="0" width="0.8128" layer="16"/>
+<wire x1="99.06" y1="0" x2="76.2" y2="0" width="0.8128" layer="16"/>
+<wire x1="102.87" y1="30.48" x2="102.87" y2="25.4" width="0.8128" layer="16"/>
+<wire x1="100.33" y1="12.7" x2="100.33" y2="1.27" width="0.8128" layer="16"/>
+<wire x1="76.2" y1="0" x2="73.66" y2="2.54" width="0.8128" layer="16"/>
+<wire x1="73.66" y1="2.54" x2="25.4" y2="2.54" width="0.8128" layer="16"/>
+<wire x1="25.4" y1="2.54" x2="20.32" y2="7.62" width="0.8128" layer="16"/>
+<wire x1="20.32" y1="7.62" x2="17.78" y2="7.62" width="0.8128" layer="16"/>
+<wire x1="17.78" y1="7.62" x2="12.7" y2="7.62" width="0.8128" layer="16"/>
+<wire x1="12.7" y1="7.62" x2="10.2" y2="5.12" width="0.8128" layer="16"/>
+<wire x1="10.2" y1="5.12" x2="10.16" y2="5.12" width="0.8128" layer="16"/>
+<wire x1="10.16" y1="63.54" x2="17.78" y2="66.04" width="0" layer="19" extent="1-1"/>
+<wire x1="17.78" y1="36.83" x2="10.16" y2="63.54" width="0" layer="19" extent="1-1"/>
+<wire x1="10.16" y1="34.33" x2="17.78" y2="36.83" width="0" layer="19" extent="1-1"/>
+<wire x1="12.7" y1="7.62" x2="10.16" y2="34.33" width="0" layer="19" extent="16-16"/>
+</signal>
 </signals>

Commit message: pcb
Parts:
- moved E$43 22.9 mm to (80.0, 92.7)
- moved E$37 1.80 mm to (90.2, 91.4)
- moved E$39 1.80 mm to (90.2, 94.0)
Connections:
- removed net S$60: E$102.1, E$103.C, E$14.1, E$14.7, E$18.1, E$19.C, E$2.1, E$2.7, E$26.1, E$26.7, E$30.1, E$31.C, E$44.1, E$45.2, E$46.2, E$47.2, E$48.2, E$49.2, E$7.1, E$74.1, E$74.7, E$78.1, E$79.C, E$86.1, E$86.7, E$9.C, E$90.1, E$91.C, E$98.1, E$98.7
- new net S$50: E$37.C, E$43.2
- net S$49: now also E$37.A, E$39.A
- net S$5: now also E$102.1, E$103.C, E$14.1, E$14.7, E$18.1, E$19.C, E$2.1, E$2.7, E$26.1, E$26.7, E$30.1, E$31.C, E$43.1, E$44.1, E$45.2, E$46.2, E$47.2, E$48.2, E$49.2, E$7.1, E$74.1, E$74.7, E$78.1, E$79.C, E$86.1, E$86.7, E$9.C, E$90.1, E$91.C, E$98.1, E$98.7
Routing:
- net S$5: track 22.9 -> 447.6 mm
- net S$60: track 392.4 -> 0.00 mm
- net S$49: track 218.5 -> 300.0 mm

Commit message: pcb
Parts:
- moved E$43 9.25 mm to (71.1, 90.2)
- moved E$37 1.27 mm to (90.2, 90.2)
Routing:
- net S$50: track 0.00 -> 15.0 mm
- net S$5: track 447.6 -> 452.5 mm
- net S$49: track 300.0 -> 302.5 mm
Changed lines of the file:
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@@
 <attribute name="VALUE" x="39.243" y="86.106" size="1.27" layer="27" ratio="10" rot="R90"/>
 </element>
-<element name="E$37" library="diode" library_urn="urn:adsk.eagle:library:210" package="DO34-7" package3d_urn="urn:adsk.eagle:package:43348/1" value="" x="90.17" y="91.44">
-<attribute name="NAME" x="88.646" y="92.583" size="1.27" layer="25" ratio="10"/>
-<attribute name="VALUE" x="88.646" y="89.027" size="1.27" layer="27" ratio="10"/>
+<element name="E$37" library="diode" library_urn="urn:adsk.eagle:library:210" package="DO34-7" package3d_urn="urn:adsk.eagle:package:43348/1" value="" x="90.17" y="90.17">
+<attribute name="NAME" x="88.646" y="91.313" size="1.27" layer="25" ratio="10"/>
+<attribute name="VALUE" x="88.646" y="87.757" size="1.27" layer="27" ratio="10"/>
 </element>
 <element name="E$38" library="con-molex" library_urn="urn:adsk.eagle:library:165" package="22-23-2021" value="" x="39.37" y="93.98" rot="R180">
@@
 <attribute name="VALUE" x="88.646" y="91.567" size="1.27" layer="27" ratio="10"/>
 </element>
-<element name="E$43" library="con-molex" library_urn="urn:adsk.eagle:library:165" package="22-23-2021" value="" x="80.01" y="92.71">
-<attribute name="NAME" x="77.47" y="96.52" size="1.016" layer="25" ratio="10"/>
-<attribute name="VALUE" x="77.47" y="87.63" size="1.016" layer="27" ratio="10"/>
+<element name="E$43" library="con-molex" library_urn="urn:adsk.eagle:library:165" package="22-23-2021" value="" x="71.12" y="90.17">
+<attribute name="NAME" x="68.58" y="93.98" size="1.016" layer="25" ratio="10"/>
+<attribute name="VALUE" x="68.58" y="85.09" size="1.016" layer="27" ratio="10"/>
 </element>
 <element name="E$44" library="con-wago-500" library_urn="urn:adsk.eagle:library:195" package="W237-102" package3d_urn="urn:adsk.eagle:package:10688/1" value="" x="99.06" y="87.63" rot="R90">
@@
 <wire x1="63.5" y1="93.98" x2="66.04" y2="93.98" width="0.8128" layer="16"/>
 <wire x1="66.04" y1="93.98" x2="67.31" y2="92.71" width="0.8128" layer="16"/>
-<wire x1="67.31" y1="92.71" x2="67.31" y2="90.17" width="0.8128" layer="16"/>
-<wire x1="67.31" y1="90.17" x2="67.945" y2="89.535" width="0.8128" layer="16"/>
-<wire x1="77.47" y1="90.17" x2="82.55" y2="90.17" width="0.8128" layer="16"/>
-<wire x1="67.945" y1="89.535" x2="76.835" y2="89.535" width="0.8128" layer="16"/>
-<wire x1="76.835" y1="89.535" x2="77.47" y2="90.17" width="0.8128" layer="16"/>
+<wire x1="67.31" y1="92.71" x2="67.31" y2="88.9" width="0.8128" layer="16"/>
+<wire x1="78.74" y1="90.17" x2="82.55" y2="90.17" width="0.8128" layer="16"/>
 <wire x1="82.55" y1="90.17" x2="87.63" y2="85.09" width="0.8128" layer="16"/>
 <wire x1="87.63" y1="85.09" x2="90.17" y2="85.09" width="0.8128" layer="16"/>
 <contactref element="E$43" pad="1"/>
-<wire x1="78.74" y1="92.71" x2="63.5" y2="93.98" width="0" layer="19" extent="1-16"/>
+<wire x1="67.31" y1="88.9" x2="68.58" y2="87.63" width="0.8128" layer="16"/>
+<wire x1="68.58" y1="87.63" x2="69.85" y2="87.63" width="0.8128" layer="16"/>
+<wire x1="69.85" y1="87.63" x2="76.2" y2="87.63" width="0.8128" layer="16"/>
+<wire x1="76.2" y1="87.63" x2="78.74" y2="90.17" width="0.8128" layer="16"/>
+<wire x1="69.85" y1="90.17" x2="69.85" y2="87.63" width="0.8128" layer="16"/>
 </signal>
 <signal name="S$33">
@@
 <contactref element="E$2" pad="8"/>
 <contactref element="E$48" pad="1"/>
-<wire x1="92.71" y1="87.63" x2="96.52" y2="87.63" width="0.8128" layer="16"/>
+<wire x1="92.71" y1="87.63" x2="93.98" y2="87.63" width="0.8128" layer="16"/>
+<wire x1="93.98" y1="87.63" x2="96.52" y2="87.63" width="0.8128" layer="16"/>
 <wire x1="99.06" y1="90.17" x2="100.29" y2="90.17" width="0.8128" layer="16"/>
 <wire x1="100.29" y1="90.17" x2="100.33" y2="90.13" width="0.8128" layer="16"/>
@@
 <wire x1="12.66" y1="66.04" x2="17.78" y2="66.04" width="0.8128" layer="16"/>
 <contactref element="E$37" pad="A"/>
-<wire x1="92.71" y1="87.63" x2="93.98" y2="91.44" width="0" layer="19" extent="1-16"/>
 <contactref element="E$39" pad="A"/>
-<wire x1="93.98" y1="91.44" x2="93.98" y2="93.98" width="0" layer="19" extent="1-16"/>
+<wire x1="93.98" y1="90.17" x2="93.98" y2="87.63" width="0.8128" layer="16"/>
+<wire x1="93.98" y1="90.17" x2="93.98" y2="93.98" width="0" layer="19" extent="1-1"/>
 </signal>
 <signal name="S$50">
 <contactref element="E$37" pad="C"/>
 <contactref element="E$43" pad="2"/>
-<wire x1="81.28" y1="92.71" x2="86.36" y2="91.44" width="0" layer="19" extent="1-16"/>
+<wire x1="72.39" y1="90.17" x2="76.2" y2="90.17" width="0.8128" layer="16"/>
+<wire x1="76.2" y1="90.17" x2="77.47" y2="91.44" width="0.8128" layer="16"/>
+<wire x1="83.82" y1="91.44" x2="85.09" y2="90.17" width="0.8128" layer="16"/>
+<wire x1="85.09" y1="90.17" x2="86.36" y2="90.17" width="0.8128" layer="16"/>
+<wire x1="77.47" y1="91.44" x2="83.82" y2="91.44" width="0.8128" layer="16"/>
 </signal>
 </signals>

Commit message: pcb
Routing:
- net S$6: track 469.3 -> 474.3 mm
Changed lines of the file:
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@@
 <wire x1="86.36" y1="31.115" x2="86.36" y2="16.51" width="0.8128" layer="16"/>
 <wire x1="22.225" y1="20.32" x2="22.225" y2="10.795" width="0.8128" layer="16"/>
-<wire x1="22.225" y1="10.795" x2="27.94" y2="5.08" width="0.8128" layer="16"/>
+<wire x1="22.225" y1="10.795" x2="27.305" y2="5.715" width="0.8128" layer="16"/>
 <wire x1="53.34" y1="19.05" x2="53.34" y2="30.48" width="0.8128" layer="16"/>
-<wire x1="53.34" y1="30.48" x2="53.975" y2="31.115" width="0.8128" layer="16"/>
-<wire x1="27.94" y1="5.08" x2="39.37" y2="5.08" width="0.8128" layer="16"/>
-<wire x1="39.37" y1="5.08" x2="53.34" y2="19.05" width="0.8128" layer="16"/>
-<wire x1="86.36" y1="31.115" x2="53.975" y2="31.115" width="0.8128" layer="16"/>
+<wire x1="40.005" y1="5.715" x2="53.34" y2="19.05" width="0.8128" layer="16"/>
 <contactref element="E$41" pad="5"/>
 <contactref element="E$40" pad="5"/>
@@
 <wire x1="45.72" y1="83.82" x2="48.26" y2="83.82" width="0.8128" layer="16"/>
 <wire x1="48.26" y1="83.82" x2="53.34" y2="83.82" width="0.8128" layer="16"/>
-<wire x1="45.72" y1="83.82" x2="38.1" y2="83.82" width="0.8128" layer="16"/>
+<wire x1="45.72" y1="83.82" x2="36.83" y2="83.82" width="0.8128" layer="16"/>
 <wire x1="36.83" y1="83.82" x2="35.56" y2="83.82" width="0.8128" layer="16"/>
 <wire x1="35.56" y1="83.82" x2="34.29" y2="85.09" width="0.8128" layer="16"/>
@@
 <wire x1="24.13" y1="92.71" x2="24.13" y2="91.44" width="0.8128" layer="16"/>
 <contactref element="E$28" pad="C"/>
-<wire x1="36.83" y1="83.82" x2="38.1" y2="83.82" width="0.8128" layer="16"/>
+<wire x1="27.305" y1="5.715" x2="40.005" y2="5.715" width="0.8128" layer="16"/>
+<wire x1="55.88" y1="33.02" x2="58.42" y2="33.02" width="0.8128" layer="16"/>
+<wire x1="62.23" y1="36.83" x2="72.39" y2="36.83" width="0.8128" layer="16"/>
+<wire x1="72.39" y1="36.83" x2="74.93" y2="34.29" width="0.8128" layer="16"/>
+<wire x1="74.93" y1="34.29" x2="74.93" y2="33.02" width="0.8128" layer="16"/>
+<wire x1="74.93" y1="33.02" x2="76.835" y2="31.115" width="0.8128" layer="16"/>
+<wire x1="53.34" y1="30.48" x2="55.88" y2="33.02" width="0.8128" layer="16"/>
+<wire x1="58.42" y1="33.02" x2="62.23" y2="36.83" width="0.8128" layer="16"/>
+<wire x1="76.835" y1="31.115" x2="86.36" y2="31.115" width="0.8128" layer="16"/>
 </signal>
 <signal name="S$7">

Commit message: pcb
Parts:
- added E$50: (no value), con-wago-500:W237-102
Connections:
- net S$5: now also E$50.1
Routing:
- net S$5: track 452.5 -> 460.9 mm
Changed lines of the file:
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@@
 <attribute name="VALUE" x="3.81" y="2.58" size="1.27" layer="28" ratio="10" rot="MR90"/>
+</element>
+<element name="E$50" library="con-wago-500" library_urn="urn:adsk.eagle:library:195" package="W237-102" package3d_urn="urn:adsk.eagle:package:10688/1" value="" x="77.47" y="95.25">
+<attribute name="NAME" x="73.6238" y="90.2462" size="1.27" layer="25" ratio="10"/>
+<attribute name="VALUE" x="72.43" y="87.63" size="1.27" layer="27" ratio="10"/>
 </element>
 </elements>
@@
 <wire x1="100.33" y1="85.13" x2="100.29" y2="85.09" width="0.8128" layer="16"/>
 <wire x1="100.29" y1="85.09" x2="92.71" y2="85.09" width="0.8128" layer="16"/>
-<wire x1="63.5" y1="93.98" x2="66.04" y2="93.98" width="0.8128" layer="16"/>
-<wire x1="66.04" y1="93.98" x2="67.31" y2="92.71" width="0.8128" layer="16"/>
-<wire x1="67.31" y1="92.71" x2="67.31" y2="88.9" width="0.8128" layer="16"/>
+<wire x1="67.31" y1="93.98" x2="67.31" y2="88.9" width="0.8128" layer="16"/>
 <wire x1="78.74" y1="90.17" x2="82.55" y2="90.17" width="0.8128" layer="16"/>
 <wire x1="82.55" y1="90.17" x2="87.63" y2="85.09" width="0.8128" layer="16"/>
@@
 <wire x1="76.2" y1="87.63" x2="78.74" y2="90.17" width="0.8128" layer="16"/>
 <wire x1="69.85" y1="90.17" x2="69.85" y2="87.63" width="0.8128" layer="16"/>
+<contactref element="E$50" pad="1"/>
+<wire x1="67.31" y1="93.98" x2="74.97" y2="93.98" width="0.8128" layer="16"/>
+<wire x1="63.5" y1="93.98" x2="67.31" y2="93.98" width="0.8128" layer="16"/>
 </signal>
 <signal name="S$33">
