File: Grbl_Esp32/src/custom/pcb/control board/controlBoard.brd (EAGLE design)
At the start: 17 parts

Commit message: controlBoard
Parts:
- added E$18, E$19: (no value), con-molex:70543-06
- added E$20, E$21, E$22, E$23, E$24, E$25, E$26, E$27, E$28, E$29, E$30, E$31, E$32: (no value), con-molex:70543-02
- moved E$3 1.27 mm to (44.5, 26.7)
Connections:
- new net S$1: E$13.6, E$15.6, E$18.1, E$18.2, E$19.1, E$19.2, E$2.6, E$20.2, E$21.2, E$22.2, E$23.2, E$24.2, E$25.2, E$26.2, E$27.2, E$28.1, E$29.1, E$30.1, E$31.1, E$32.1, E$9.6
- new net S$2: E$13.7, E$15.7, E$18.3, E$19.3, E$2.7, E$9.7
- new net S$3: E$13.8, E$15.8, E$18.4, E$19.4, E$2.8, E$9.8
- new net S$4: E$13.9, E$15.9, E$18.5, E$19.5, E$2.9, E$9.9
- new net S$5: E$1.1, E$12.1, E$14.1, E$20.1, E$21.1, E$8.1
- new net S$6: E$1.2, E$12.2, E$14.2, E$22.1, E$23.1, E$8.2
- new net S$7: E$1.3, E$12.3, E$14.3, E$24.1, E$25.1, E$8.3
- new net S$8: E$13.5, E$15.5, E$2.5, E$26.1, E$27.1, E$9.5
- new net S$9: E$1.8, E$12.8, E$14.8, E$28.2, E$29.2, E$30.2, E$31.2, E$32.2, E$8.8
Routing:
- net S$1: track 0.00 -> 62.8 mm
- net S$9: track 0.00 -> 25.4 mm
- net S$5: track 0.00 -> 23.9 mm
- net S$8: track 0.00 -> 21.4 mm
- net S$7: track 0.00 -> 17.6 mm
- net S$6: track 0.00 -> 16.5 mm
- net S$4: track 0.00 -> 16.5 mm
- net S$3: track 0.00 -> 16.5 mm
- net S$2: track 0.00 -> 16.5 mm

Commit message: controlBoard
Parts:
- added E$33: (no value), con-molex:70543-03
- added E$34, E$35: (no value), diode:DO34-7
- added E$36, E$37, E$38: (no value), con-wago-500:W237-102
Connections:
- new net S$10: E$13.10, E$15.10, E$2.10, E$34.A, E$9.10
Routing:
- net S$10: track 0.00 -> 21.4 mm
Changed lines of the file:
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@@
 <layer number="97" name="Info" color="7" fill="1" visible="no" active="no"/>
 <layer number="98" name="Guide" color="6" fill="1" visible="no" active="no"/>
+<layer number="99" name="SpiceOrder" color="5" fill="1" visible="no" active="no"/>
 </layers>
 <board>
@@
 <attribute name="VALUE" x="5.3975" y="68.8975" size="0.8128" layer="27" ratio="10" rot="R90"/>
 </element>
+<element name="E$33" library="con-molex" library_urn="urn:adsk.eagle:library:165" package="70543-03" value="" x="3.81" y="52.07" rot="R90">
+<attribute name="NAME" x="6.35" y="46.355" size="1.016" layer="25" ratio="10" rot="R180"/>
+<attribute name="VALUE" x="0.3175" y="47.3075" size="0.8128" layer="27" ratio="10" rot="R90"/>
+</element>
+<element name="E$34" library="diode" library_urn="urn:adsk.eagle:library:210" package="DO34-7" package3d_urn="urn:adsk.eagle:package:43348/1" value="" x="12.7" y="50.8" rot="R90">
+<attribute name="NAME" x="11.557" y="49.276" size="1.27" layer="25" ratio="10" rot="R90"/>
+<attribute name="VALUE" x="15.113" y="49.276" size="1.27" layer="27" ratio="10" rot="R90"/>
+</element>
+<element name="E$35" library="diode" library_urn="urn:adsk.eagle:library:210" package="DO34-7" package3d_urn="urn:adsk.eagle:package:43348/1" value="" x="6.35" y="39.37" rot="R90">
+<attribute name="NAME" x="5.207" y="37.846" size="1.27" layer="25" ratio="10" rot="R90"/>
+<attribute name="VALUE" x="8.763" y="37.846" size="1.27" layer="27" ratio="10" rot="R90"/>
+</element>
+<element name="E$36" library="con-wago-500" library_urn="urn:adsk.eagle:library:195" package="W237-102" package3d_urn="urn:adsk.eagle:package:10688/1" value="" x="-3.81" y="49.53" rot="R90">
+<attribute name="NAME" x="1.1938" y="45.6838" size="1.27" layer="25" ratio="10" rot="R90"/>
+<attribute name="VALUE" x="3.81" y="44.49" size="1.27" layer="27" ratio="10" rot="R90"/>
+</element>
+<element name="E$37" library="con-wago-500" library_urn="urn:adsk.eagle:library:195" package="W237-102" package3d_urn="urn:adsk.eagle:package:10688/1" value="" x="-3.81" y="41.91" rot="R90">
+<attribute name="NAME" x="1.1938" y="38.0638" size="1.27" layer="25" ratio="10" rot="R90"/>
+<attribute name="VALUE" x="3.81" y="36.87" size="1.27" layer="27" ratio="10" rot="R90"/>
+</element>
+<element name="E$38" library="con-wago-500" library_urn="urn:adsk.eagle:library:195" package="W237-102" package3d_urn="urn:adsk.eagle:package:10688/1" value="" x="1.27" y="40.64" rot="R90">
+<attribute name="NAME" x="6.2738" y="36.7938" size="1.27" layer="25" ratio="10" rot="R90"/>
+<attribute name="VALUE" x="8.89" y="35.6" size="1.27" layer="27" ratio="10" rot="R90"/>
+</element>
 </elements>
 <signals>
@@
 <wire x1="30.48" y1="73.66" x2="33.02" y2="73.66" width="0.6096" layer="16"/>
 </signal>
+<signal name="S$10">
+<contactref element="E$9" pad="10"/>
+<contactref element="E$2" pad="10"/>
+<contactref element="E$13" pad="10"/>
+<contactref element="E$15" pad="10"/>
+<contactref element="E$34" pad="A"/>
+<wire x1="12.7" y1="54.61" x2="13.97" y2="54.61" width="0.6096" layer="16"/>
+<wire x1="22.86" y1="53.34" x2="25.4" y2="53.34" width="0.6096" layer="16"/>
+<wire x1="25.4" y1="53.34" x2="27.94" y2="53.34" width="0.6096" layer="16"/>
+<wire x1="27.94" y1="53.34" x2="30.48" y2="53.34" width="0.6096" layer="16"/>
+<wire x1="30.48" y1="53.34" x2="33.02" y2="53.34" width="0.6096" layer="16"/>
+<wire x1="13.97" y1="54.61" x2="14.605" y2="55.245" width="0.6096" layer="16"/>
+<wire x1="14.605" y1="55.245" x2="20.955" y2="55.245" width="0.6096" layer="16"/>
+<wire x1="20.955" y1="55.245" x2="22.86" y2="53.34" width="0.6096" layer="16"/>
+</signal>
 </signals>

Commit message: controlBoard
Parts:
- moved E$33 5.68 mm to (8.89, 49.5)
Connections:
- new net S$11: E$33.1, E$34.C
- new net S$12: E$13.1, E$15.1, E$18.6, E$19.6, E$2.1, E$9.1
- net S$1: now also E$33.3
Routing:
- net S$12: track 0.00 -> 52.4 mm
- net S$1: track 62.8 -> 88.2 mm
- net S$11: track 0.00 -> 3.81 mm
Changed lines of the file:
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@@
 <attribute name="VALUE" x="5.3975" y="68.8975" size="0.8128" layer="27" ratio="10" rot="R90"/>
 </element>
-<element name="E$33" library="con-molex" library_urn="urn:adsk.eagle:library:165" package="70543-03" value="" x="3.81" y="52.07" rot="R90">
-<attribute name="NAME" x="6.35" y="46.355" size="1.016" layer="25" ratio="10" rot="R180"/>
-<attribute name="VALUE" x="0.3175" y="47.3075" size="0.8128" layer="27" ratio="10" rot="R90"/>
+<element name="E$33" library="con-molex" library_urn="urn:adsk.eagle:library:165" package="70543-03" value="" x="8.89" y="49.53" rot="R90">
+<attribute name="NAME" x="11.43" y="43.815" size="1.016" layer="25" ratio="10" rot="R180"/>
+<attribute name="VALUE" x="5.3975" y="44.7675" size="0.8128" layer="27" ratio="10" rot="R90"/>
 </element>
 <element name="E$34" library="diode" library_urn="urn:adsk.eagle:library:210" package="DO34-7" package3d_urn="urn:adsk.eagle:package:43348/1" value="" x="12.7" y="50.8" rot="R90">
@@
 <wire x1="16.51" y1="71.12" x2="19.05" y2="71.12" width="0.6096" layer="16"/>
 <wire x1="19.05" y1="71.12" x2="19.05" y2="66.04" width="0.6096" layer="16"/>
-<wire x1="16.51" y1="43.18" x2="16.51" y2="60.96" width="0" layer="19" extent="1-1"/>
+<contactref element="E$33" pad="3"/>
+<wire x1="10.16" y1="60.96" x2="8.89" y2="60.96" width="0.6096" layer="16"/>
+<wire x1="8.89" y1="60.96" x2="7.62" y2="59.69" width="0.6096" layer="16"/>
+<wire x1="7.62" y1="59.69" x2="7.62" y2="54.61" width="0.6096" layer="16"/>
+<wire x1="7.62" y1="54.61" x2="8.89" y2="53.34" width="0.6096" layer="16"/>
+<wire x1="8.89" y1="53.34" x2="8.89" y2="52.07" width="0.6096" layer="16"/>
+<wire x1="8.89" y1="52.07" x2="11.43" y2="52.07" width="0.6096" layer="16"/>
+<wire x1="13.97" y1="44.45" x2="15.24" y2="43.18" width="0.6096" layer="16"/>
+<wire x1="15.24" y1="43.18" x2="16.51" y2="43.18" width="0.6096" layer="16"/>
+<wire x1="11.43" y1="52.07" x2="13.97" y2="49.53" width="0.6096" layer="16"/>
+<wire x1="13.97" y1="49.53" x2="13.97" y2="44.45" width="0.6096" layer="16"/>
 </signal>
 <signal name="S$2">
@@
 <wire x1="20.955" y1="55.245" x2="22.86" y2="53.34" width="0.6096" layer="16"/>
 </signal>
+<signal name="S$11">
+<contactref element="E$33" pad="1"/>
+<contactref element="E$34" pad="C"/>
+<wire x1="8.89" y1="46.99" x2="12.7" y2="46.99" width="0.6096" layer="16"/>
+</signal>
+<signal name="S$12">
+<contactref element="E$18" pad="6"/>
+<contactref element="E$19" pad="6"/>
+<contactref element="E$15" pad="1"/>
+<contactref element="E$13" pad="1"/>
+<contactref element="E$9" pad="1"/>
+<contactref element="E$2" pad="1"/>
+<wire x1="25.4" y1="30.48" x2="27.94" y2="30.48" width="0.6096" layer="16"/>
+<wire x1="27.94" y1="30.48" x2="30.48" y2="30.48" width="0.6096" layer="16"/>
+<wire x1="30.48" y1="30.48" x2="33.02" y2="30.48" width="0.6096" layer="16"/>
+<wire x1="33.02" y1="30.48" x2="35.56" y2="30.48" width="0.6096" layer="16"/>
+<wire x1="35.56" y1="30.48" x2="36.83" y2="31.75" width="0.6096" layer="16"/>
+<wire x1="36.83" y1="31.75" x2="36.83" y2="50.8" width="0.6096" layer="16"/>
+<wire x1="36.83" y1="50.8" x2="35.56" y2="52.07" width="0.6096" layer="16"/>
+<wire x1="21.59" y1="52.07" x2="20.32" y2="53.34" width="0.6096" layer="16"/>
+<wire x1="20.32" y1="53.34" x2="19.05" y2="53.34" width="0.6096" layer="16"/>
+<wire x1="35.56" y1="52.07" x2="21.59" y2="52.07" width="0.6096" layer="16"/>
+<wire x1="19.05" y1="53.34" x2="16.51" y2="53.34" width="0.6096" layer="16"/>
+</signal>
 </signals>

Commit message: controlBoard
Parts:
- added E$39: (no value), con-wago-500:W237-102
- moved E$38 7.62 mm to (8.89, 40.6)
- moved E$36 6.48 mm to (2.54, 50.8), turned to 270 degrees
- moved E$35 6.35 mm to (6.35, 45.7)
- moved E$37 6.35 mm to (2.54, 41.9), turned to 270 degrees
Connections:
- new net S$13: E$33.2, E$35.A, E$38.2
- new net S$14: E$35.C, E$38.1
Changed lines of the file:
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@@
 <attribute name="VALUE" x="15.113" y="49.276" size="1.27" layer="27" ratio="10" rot="R90"/>
 </element>
-<element name="E$35" library="diode" library_urn="urn:adsk.eagle:library:210" package="DO34-7" package3d_urn="urn:adsk.eagle:package:43348/1" value="" x="6.35" y="39.37" rot="R90">
-<attribute name="NAME" x="5.207" y="37.846" size="1.27" layer="25" ratio="10" rot="R90"/>
-<attribute name="VALUE" x="8.763" y="37.846" size="1.27" layer="27" ratio="10" rot="R90"/>
-</element>
-<element name="E$36" library="con-wago-500" library_urn="urn:adsk.eagle:library:195" package="W237-102" package3d_urn="urn:adsk.eagle:package:10688/1" value="" x="-3.81" y="49.53" rot="R90">
-<attribute name="NAME" x="1.1938" y="45.6838" size="1.27" layer="25" ratio="10" rot="R90"/>
-<attribute name="VALUE" x="3.81" y="44.49" size="1.27" layer="27" ratio="10" rot="R90"/>
-</element>
-<element name="E$37" library="con-wago-500" library_urn="urn:adsk.eagle:library:195" package="W237-102" package3d_urn="urn:adsk.eagle:package:10688/1" value="" x="-3.81" y="41.91" rot="R90">
-<attribute name="NAME" x="1.1938" y="38.0638" size="1.27" layer="25" ratio="10" rot="R90"/>
-<attribute name="VALUE" x="3.81" y="36.87" size="1.27" layer="27" ratio="10" rot="R90"/>
-</element>
-<element name="E$38" library="con-wago-500" library_urn="urn:adsk.eagle:library:195" package="W237-102" package3d_urn="urn:adsk.eagle:package:10688/1" value="" x="1.27" y="40.64" rot="R90">
-<attribute name="NAME" x="6.2738" y="36.7938" size="1.27" layer="25" ratio="10" rot="R90"/>
-<attribute name="VALUE" x="8.89" y="35.6" size="1.27" layer="27" ratio="10" rot="R90"/>
+<element name="E$35" library="diode" library_urn="urn:adsk.eagle:library:210" package="DO34-7" package3d_urn="urn:adsk.eagle:package:43348/1" value="" x="6.35" y="45.72" rot="R90">
+<attribute name="NAME" x="5.207" y="44.196" size="1.27" layer="25" ratio="10" rot="R90"/>
+<attribute name="VALUE" x="8.763" y="44.196" size="1.27" layer="27" ratio="10" rot="R90"/>
+</element>
+<element name="E$36" library="con-wago-500" library_urn="urn:adsk.eagle:library:195" package="W237-102" package3d_urn="urn:adsk.eagle:package:10688/1" value="" x="2.54" y="50.8" rot="R270">
+<attribute name="NAME" x="-2.4638" y="54.6462" size="1.27" layer="25" ratio="10" rot="R270"/>
+<attribute name="VALUE" x="-5.08" y="55.84" size="1.27" layer="27" ratio="10" rot="R270"/>
+</element>
+<element name="E$37" library="con-wago-500" library_urn="urn:adsk.eagle:library:195" package="W237-102" package3d_urn="urn:adsk.eagle:package:10688/1" value="" x="2.54" y="41.91" rot="R270">
+<attribute name="NAME" x="-2.4638" y="45.7562" size="1.27" layer="25" ratio="10" rot="R270"/>
+<attribute name="VALUE" x="-5.08" y="46.95" size="1.27" layer="27" ratio="10" rot="R270"/>
+</element>
+<element name="E$38" library="con-wago-500" library_urn="urn:adsk.eagle:library:195" package="W237-102" package3d_urn="urn:adsk.eagle:package:10688/1" value="" x="8.89" y="40.64" rot="R90">
+<attribute name="NAME" x="13.8938" y="36.7938" size="1.27" layer="25" ratio="10" rot="R90"/>
+<attribute name="VALUE" x="16.51" y="35.6" size="1.27" layer="27" ratio="10" rot="R90"/>
+</element>
+<element name="E$39" library="con-wago-500" library_urn="urn:adsk.eagle:library:195" package="W237-102" package3d_urn="urn:adsk.eagle:package:10688/1" value="" x="2.54" y="33.02" rot="R270">
+<attribute name="NAME" x="-2.4638" y="36.8662" size="1.27" layer="25" ratio="10" rot="R270"/>
+<attribute name="VALUE" x="-5.08" y="38.06" size="1.27" layer="27" ratio="10" rot="R270"/>
 </element>
 </elements>
@@
 <wire x1="19.05" y1="53.34" x2="16.51" y2="53.34" width="0.6096" layer="16"/>
 </signal>
+<signal name="S$13">
+<contactref element="E$35" pad="A"/>
+<contactref element="E$33" pad="2"/>
+<wire x1="8.89" y1="49.53" x2="6.35" y2="49.53" width="0" layer="19" extent="1-16"/>
+<contactref element="E$38" pad="2"/>
+<wire x1="10.16" y1="43.14" x2="6.35" y2="49.53" width="0" layer="19" extent="1-16"/>
+</signal>
+<signal name="S$14">
+<contactref element="E$38" pad="1"/>
+<contactref element="E$35" pad="C"/>
+<wire x1="6.35" y1="41.91" x2="10.16" y2="38.14" width="0" layer="19" extent="1-16"/>
+</signal>
 </signals>

Commit message: controlBoard
Connections:
- net S$1: now also E$37.2, E$39.1
- net S$12: now also E$39.2
- net S$13: now also E$36.1
- net S$14: now also E$36.2, E$37.1
Routing:
- net S$12: track 52.4 -> 76.5 mm
- net S$1: track 88.2 -> 107.9 mm
- net S$13: track 0.00 -> 19.4 mm
- net S$14: track 0.00 -> 16.9 mm
Changed lines of the file:
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@@
 <wire x1="11.43" y1="52.07" x2="13.97" y2="49.53" width="0.6096" layer="16"/>
 <wire x1="13.97" y1="49.53" x2="13.97" y2="44.45" width="0.6096" layer="16"/>
+<contactref element="E$37" pad="2"/>
+<contactref element="E$39" pad="1"/>
+<wire x1="1.27" y1="39.41" x2="1.27" y2="35.52" width="0.6096" layer="16"/>
+<wire x1="1.27" y1="35.52" x2="12.66" y2="35.52" width="0.6096" layer="16"/>
+<wire x1="13.97" y1="36.83" x2="16.51" y2="36.83" width="0.6096" layer="16"/>
+<wire x1="12.66" y1="35.52" x2="13.97" y2="36.83" width="0.6096" layer="16"/>
 </signal>
 <signal name="S$2">
@@
 <wire x1="35.56" y1="52.07" x2="21.59" y2="52.07" width="0.6096" layer="16"/>
 <wire x1="19.05" y1="53.34" x2="16.51" y2="53.34" width="0.6096" layer="16"/>
+<contactref element="E$39" pad="2"/>
+<wire x1="1.27" y1="30.52" x2="25.36" y2="30.52" width="0.6096" layer="16"/>
+<wire x1="25.36" y1="30.52" x2="25.4" y2="30.48" width="0.6096" layer="16"/>
 </signal>
 <signal name="S$13">
 <contactref element="E$35" pad="A"/>
 <contactref element="E$33" pad="2"/>
-<wire x1="8.89" y1="49.53" x2="6.35" y2="49.53" width="0" layer="19" extent="1-16"/>
 <contactref element="E$38" pad="2"/>
-<wire x1="10.16" y1="43.14" x2="6.35" y2="49.53" width="0" layer="19" extent="1-16"/>
+<wire x1="8.89" y1="49.53" x2="6.35" y2="49.53" width="0.6096" layer="16"/>
+<wire x1="6.35" y1="49.53" x2="6.35" y2="45.72" width="0.6096" layer="16"/>
+<wire x1="8.93" y1="43.14" x2="10.16" y2="43.14" width="0.6096" layer="16"/>
+<wire x1="6.35" y1="45.72" x2="8.93" y2="43.14" width="0.6096" layer="16"/>
+<contactref element="E$36" pad="1"/>
+<wire x1="1.27" y1="53.3" x2="5.12" y2="53.3" width="0.6096" layer="16"/>
+<wire x1="5.12" y1="53.3" x2="6.35" y2="52.07" width="0.6096" layer="16"/>
+<wire x1="6.35" y1="52.07" x2="6.35" y2="49.53" width="0.6096" layer="16"/>
 </signal>
 <signal name="S$14">
 <contactref element="E$38" pad="1"/>
 <contactref element="E$35" pad="C"/>
-<wire x1="6.35" y1="41.91" x2="10.16" y2="38.14" width="0" layer="19" extent="1-16"/>
+<wire x1="6.35" y1="41.91" x2="6.35" y2="39.37" width="0.6096" layer="16"/>
+<wire x1="7.62" y1="38.1" x2="6.35" y2="39.37" width="0.6096" layer="16"/>
+<wire x1="10.16" y1="38.14" x2="10.12" y2="38.1" width="0.6096" layer="16"/>
+<wire x1="10.12" y1="38.1" x2="7.62" y2="38.1" width="0.6096" layer="16"/>
+<contactref element="E$37" pad="1"/>
+<contactref element="E$36" pad="2"/>
+<wire x1="1.27" y1="48.3" x2="1.27" y2="44.41" width="0.6096" layer="16"/>
+<wire x1="1.27" y1="44.41" x2="3.77" y2="41.91" width="0.6096" layer="16"/>
+<wire x1="3.77" y1="41.91" x2="6.35" y2="41.91" width="0.6096" layer="16"/>
 </signal>
 </signals>

Commit message: controlBoard
Parts:
- added E$40: (no value), con-wago-500:W237-102
Connections:
- net S$1: now also E$40.2
- net S$12: now also E$40.1
Changed lines of the file:
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@@
 <attribute name="VALUE" x="-5.08" y="38.06" size="1.27" layer="27" ratio="10" rot="R270"/>
+</element>
+<element name="E$40" library="con-wago-500" library_urn="urn:adsk.eagle:library:195" package="W237-102" package3d_urn="urn:adsk.eagle:package:10688/1" value="" x="8.89" y="33.02" rot="R90">
+<attribute name="NAME" x="13.8938" y="29.1738" size="1.27" layer="25" ratio="10" rot="R90"/>
+<attribute name="VALUE" x="16.51" y="27.98" size="1.27" layer="27" ratio="10" rot="R90"/>
 </element>
 </elements>
@@
 <contactref element="E$39" pad="1"/>
 <wire x1="1.27" y1="39.41" x2="1.27" y2="35.52" width="0.6096" layer="16"/>
-<wire x1="1.27" y1="35.52" x2="12.66" y2="35.52" width="0.6096" layer="16"/>
+<wire x1="1.27" y1="35.52" x2="7.62" y2="35.52" width="0.6096" layer="16"/>
+<wire x1="10.16" y1="35.52" x2="12.66" y2="35.52" width="0.6096" layer="16"/>
 <wire x1="13.97" y1="36.83" x2="16.51" y2="36.83" width="0.6096" layer="16"/>
 <wire x1="12.66" y1="35.52" x2="13.97" y2="36.83" width="0.6096" layer="16"/>
+<contactref element="E$40" pad="2"/>
+<wire x1="10.16" y1="35.52" x2="7.62" y2="35.52" width="0.6096" layer="16"/>
 </signal>
 <signal name="S$2">
@@
 <wire x1="19.05" y1="53.34" x2="16.51" y2="53.34" width="0.6096" layer="16"/>
 <contactref element="E$39" pad="2"/>
-<wire x1="1.27" y1="30.52" x2="25.36" y2="30.52" width="0.6096" layer="16"/>
+<wire x1="1.27" y1="30.52" x2="7.62" y2="30.52" width="0.6096" layer="16"/>
+<wire x1="10.16" y1="30.52" x2="25.36" y2="30.52" width="0.6096" layer="16"/>
 <wire x1="25.36" y1="30.52" x2="25.4" y2="30.48" width="0.6096" layer="16"/>
+<contactref element="E$40" pad="1"/>
+<wire x1="10.16" y1="30.52" x2="7.62" y2="30.52" width="0.6096" layer="16"/>
 </signal>
 <signal name="S$13">

Commit message: controlBoard
Parts:
- moved E$36 2.54 mm to (2.54, 53.3)
- moved E$37 1.27 mm to (2.54, 43.2)
Routing:
- net S$14: track 16.9 -> 18.7 mm
- net S$13: track 19.4 -> 21.2 mm
- net S$1: track 107.9 -> 109.2 mm
Changed lines of the file:
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@@
 <attribute name="VALUE" x="8.763" y="44.196" size="1.27" layer="27" ratio="10" rot="R90"/>
 </element>
-<element name="E$36" library="con-wago-500" library_urn="urn:adsk.eagle:library:195" package="W237-102" package3d_urn="urn:adsk.eagle:package:10688/1" value="" x="2.54" y="50.8" rot="R270">
-<attribute name="NAME" x="-2.4638" y="54.6462" size="1.27" layer="25" ratio="10" rot="R270"/>
-<attribute name="VALUE" x="-5.08" y="55.84" size="1.27" layer="27" ratio="10" rot="R270"/>
-</element>
-<element name="E$37" library="con-wago-500" library_urn="urn:adsk.eagle:library:195" package="W237-102" package3d_urn="urn:adsk.eagle:package:10688/1" value="" x="2.54" y="41.91" rot="R270">
-<attribute name="NAME" x="-2.4638" y="45.7562" size="1.27" layer="25" ratio="10" rot="R270"/>
-<attribute name="VALUE" x="-5.08" y="46.95" size="1.27" layer="27" ratio="10" rot="R270"/>
+<element name="E$36" library="con-wago-500" library_urn="urn:adsk.eagle:library:195" package="W237-102" package3d_urn="urn:adsk.eagle:package:10688/1" value="" x="2.54" y="53.34" rot="R270">
+<attribute name="NAME" x="-2.4638" y="57.1862" size="1.27" layer="25" ratio="10" rot="R270"/>
+<attribute name="VALUE" x="-5.08" y="58.38" size="1.27" layer="27" ratio="10" rot="R270"/>
+</element>
+<element name="E$37" library="con-wago-500" library_urn="urn:adsk.eagle:library:195" package="W237-102" package3d_urn="urn:adsk.eagle:package:10688/1" value="" x="2.54" y="43.18" rot="R270">
+<attribute name="NAME" x="-2.4638" y="47.0262" size="1.27" layer="25" ratio="10" rot="R270"/>
+<attribute name="VALUE" x="-5.08" y="48.22" size="1.27" layer="27" ratio="10" rot="R270"/>
 </element>
 <element name="E$38" library="con-wago-500" library_urn="urn:adsk.eagle:library:195" package="W237-102" package3d_urn="urn:adsk.eagle:package:10688/1" value="" x="8.89" y="40.64" rot="R90">
@@
 <contactref element="E$37" pad="2"/>
 <contactref element="E$39" pad="1"/>
-<wire x1="1.27" y1="39.41" x2="1.27" y2="35.52" width="0.6096" layer="16"/>
-<wire x1="1.27" y1="35.52" x2="7.62" y2="35.52" width="0.6096" layer="16"/>
+<wire x1="1.27" y1="40.68" x2="1.27" y2="35.52" width="0.6096" layer="16"/>
+<wire x1="1.27" y1="35.52" x2="10.16" y2="35.52" width="0.6096" layer="16"/>
 <wire x1="10.16" y1="35.52" x2="12.66" y2="35.52" width="0.6096" layer="16"/>
 <wire x1="13.97" y1="36.83" x2="16.51" y2="36.83" width="0.6096" layer="16"/>
 <wire x1="12.66" y1="35.52" x2="13.97" y2="36.83" width="0.6096" layer="16"/>
 <contactref element="E$40" pad="2"/>
-<wire x1="10.16" y1="35.52" x2="7.62" y2="35.52" width="0.6096" layer="16"/>
 </signal>
 <signal name="S$2">
@@
 <wire x1="6.35" y1="45.72" x2="8.93" y2="43.14" width="0.6096" layer="16"/>
 <contactref element="E$36" pad="1"/>
-<wire x1="1.27" y1="53.3" x2="5.12" y2="53.3" width="0.6096" layer="16"/>
-<wire x1="5.12" y1="53.3" x2="6.35" y2="52.07" width="0.6096" layer="16"/>
-<wire x1="6.35" y1="52.07" x2="6.35" y2="49.53" width="0.6096" layer="16"/>
+<wire x1="3.85" y1="55.84" x2="1.27" y2="55.84" width="0.6096" layer="16"/>
+<wire x1="6.35" y1="53.34" x2="3.85" y2="55.84" width="0.6096" layer="16"/>
+<wire x1="6.35" y1="53.34" x2="6.35" y2="49.53" width="0.6096" layer="16"/>
 </signal>
 <signal name="S$14">
@@
 <contactref element="E$37" pad="1"/>
 <contactref element="E$36" pad="2"/>
-<wire x1="1.27" y1="48.3" x2="1.27" y2="44.41" width="0.6096" layer="16"/>
-<wire x1="1.27" y1="44.41" x2="3.77" y2="41.91" width="0.6096" layer="16"/>
-<wire x1="3.77" y1="41.91" x2="6.35" y2="41.91" width="0.6096" layer="16"/>
+<wire x1="1.27" y1="50.84" x2="1.27" y2="45.68" width="0.6096" layer="16"/>
+<wire x1="5.04" y1="41.91" x2="1.27" y2="45.68" width="0.6096" layer="16"/>
+<wire x1="5.04" y1="41.91" x2="6.35" y2="41.91" width="0.6096" layer="16"/>
 </signal>
 </signals>
