File: Grbl_Esp32/src/custom/pcb/control board/controlBoard.brd (EAGLE design)
At the start: 40 parts

Commit message: controlBoard
Parts:
- removed E$3: (no value), con-lstb:MA10-1
- added E$41: (no value), con-lsta:FE06
- added E$42: (no value), con-lsta:FE07
Connections:
- new net S$15: E$11.10, E$17.10, E$41.1, E$5.10, E$7.10
- new net S$16: E$10.1, E$16.1, E$4.1, E$41.2, E$6.1
- new net S$17: E$10.8, E$16.8, E$4.8, E$41.3, E$6.8
- new net S$18: E$10.2, E$16.2, E$4.2, E$41.4, E$6.2
- net S$1: now also E$10.3, E$16.3, E$4.3, E$4.9, E$41.6, E$6.3
- net S$12: now also E$41.5
Routing:
- net S$1: track 109.2 -> 178.6 mm
- net S$12: track 76.5 -> 144.7 mm
- net S$17: track 0.00 -> 34.1 mm
- net S$15: track 0.00 -> 31.5 mm
- net S$16: track 0.00 -> 28.2 mm
- net S$18: track 0.00 -> 22.4 mm
Changed lines of the file:
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@@
 <attribute name="VALUE" x="35.941" y="43.18" size="1.27" layer="27" ratio="10" rot="R90"/>
-</element>
-<element name="E$3" library="con-lstb" library_urn="urn:adsk.eagle:library:162" package="MA10-1" package3d_urn="urn:adsk.eagle:package:8346/1" value="" x="44.45" y="26.67" rot="R180">
-<attribute name="NAME" x="57.15" y="25.019" size="1.27" layer="25" ratio="10" rot="R180"/>
-<attribute name="VALUE" x="43.18" y="29.591" size="1.27" layer="27" ratio="10" rot="R180"/>
 </element>
 <element name="E$4" library="con-lstb" library_urn="urn:adsk.eagle:library:162" package="MA09-1" package3d_urn="urn:adsk.eagle:package:8350/1" value="" x="55.88" y="66.04" rot="R90">
@@
 <attribute name="NAME" x="13.8938" y="29.1738" size="1.27" layer="25" ratio="10" rot="R90"/>
 <attribute name="VALUE" x="16.51" y="27.98" size="1.27" layer="27" ratio="10" rot="R90"/>
+</element>
+<element name="E$41" library="con-lsta" library_urn="urn:adsk.eagle:library:161" package="FE06" package3d_urn="urn:adsk.eagle:package:8191/1" value="" x="74.93" y="58.42" rot="R180">
+<attribute name="NAME" x="78.74" y="56.769" size="1.27" layer="25" ratio="10" rot="R180"/>
+<attribute name="VALUE" x="82.55" y="61.341" size="1.27" layer="27" ratio="10" rot="R180"/>
+</element>
+<element name="E$42" library="con-lsta" library_urn="urn:adsk.eagle:library:161" package="FE07" package3d_urn="urn:adsk.eagle:package:8223/1" value="" x="81.28" y="38.1" rot="R90">
+<attribute name="NAME" x="79.629" y="33.02" size="1.27" layer="25" ratio="10" rot="R90"/>
+<attribute name="VALUE" x="84.201" y="30.48" size="1.27" layer="27" ratio="10" rot="R90"/>
 </element>
 </elements>
@@
 <wire x1="12.66" y1="35.52" x2="13.97" y2="36.83" width="0.6096" layer="16"/>
 <contactref element="E$40" pad="2"/>
+<contactref element="E$4" pad="9"/>
+<contactref element="E$4" pad="3"/>
+<wire x1="19.05" y1="71.12" x2="20.32" y2="71.12" width="0.6096" layer="16"/>
+<wire x1="20.32" y1="71.12" x2="21.59" y2="72.39" width="0.6096" layer="16"/>
+<wire x1="53.34" y1="76.2" x2="55.88" y2="76.2" width="0.6096" layer="16"/>
+<wire x1="21.59" y1="72.39" x2="52.07" y2="72.39" width="0.6096" layer="16"/>
+<wire x1="55.88" y1="60.96" x2="53.34" y2="60.96" width="0.6096" layer="16"/>
+<wire x1="53.34" y1="60.96" x2="52.07" y2="62.23" width="0.6096" layer="16"/>
+<wire x1="52.07" y1="62.23" x2="52.07" y2="72.39" width="0.6096" layer="16"/>
+<wire x1="52.07" y1="72.39" x2="52.07" y2="74.93" width="0.6096" layer="16"/>
+<wire x1="52.07" y1="74.93" x2="53.34" y2="76.2" width="0.6096" layer="16"/>
+<contactref element="E$16" pad="3"/>
+<contactref element="E$41" pad="6"/>
+<contactref element="E$10" pad="3"/>
+<contactref element="E$6" pad="3"/>
+<wire x1="68.58" y1="58.42" x2="68.58" y2="59.69" width="0.6096" layer="16"/>
+<wire x1="68.58" y1="59.69" x2="67.31" y2="60.96" width="0.6096" layer="16"/>
+<wire x1="67.31" y1="60.96" x2="63.5" y2="60.96" width="0.6096" layer="16"/>
+<wire x1="63.5" y1="60.96" x2="60.96" y2="60.96" width="0.6096" layer="16"/>
+<wire x1="60.96" y1="60.96" x2="58.42" y2="60.96" width="0.6096" layer="16"/>
+<wire x1="58.42" y1="60.96" x2="55.88" y2="60.96" width="0.6096" layer="16"/>
 </signal>
 <signal name="S$2">
@@
 <wire x1="30.48" y1="30.48" x2="33.02" y2="30.48" width="0.6096" layer="16"/>
 <wire x1="33.02" y1="30.48" x2="35.56" y2="30.48" width="0.6096" layer="16"/>
-<wire x1="35.56" y1="30.48" x2="36.83" y2="31.75" width="0.6096" layer="16"/>
-<wire x1="36.83" y1="31.75" x2="36.83" y2="50.8" width="0.6096" layer="16"/>
-<wire x1="36.83" y1="50.8" x2="35.56" y2="52.07" width="0.6096" layer="16"/>
+<wire x1="36.83" y1="31.75" x2="35.56" y2="30.48" width="0.6096" layer="16"/>
 <wire x1="21.59" y1="52.07" x2="20.32" y2="53.34" width="0.6096" layer="16"/>
 <wire x1="20.32" y1="53.34" x2="19.05" y2="53.34" width="0.6096" layer="16"/>
-<wire x1="35.56" y1="52.07" x2="21.59" y2="52.07" width="0.6096" layer="16"/>
+<wire x1="36.83" y1="52.07" x2="21.59" y2="52.07" width="0.6096" layer="16"/>
 <wire x1="19.05" y1="53.34" x2="16.51" y2="53.34" width="0.6096" layer="16"/>
 <contactref element="E$39" pad="2"/>
-<wire x1="1.27" y1="30.52" x2="7.62" y2="30.52" width="0.6096" layer="16"/>
+<wire x1="1.27" y1="30.52" x2="10.16" y2="30.52" width="0.6096" layer="16"/>
 <wire x1="10.16" y1="30.52" x2="25.36" y2="30.52" width="0.6096" layer="16"/>
 <wire x1="25.36" y1="30.52" x2="25.4" y2="30.48" width="0.6096" layer="16"/>
 <contactref element="E$40" pad="1"/>
-<wire x1="10.16" y1="30.52" x2="7.62" y2="30.52" width="0.6096" layer="16"/>
+<contactref element="E$41" pad="5"/>
+<wire x1="36.83" y1="52.07" x2="36.83" y2="69.85" width="0.6096" layer="16"/>
+<wire x1="36.83" y1="69.85" x2="38.1" y2="71.12" width="0.6096" layer="16"/>
+<wire x1="49.53" y1="71.12" x2="50.8" y2="69.85" width="0.6096" layer="16"/>
+<wire x1="50.8" y1="69.85" x2="50.8" y2="60.96" width="0.6096" layer="16"/>
+<wire x1="50.8" y1="60.96" x2="52.07" y2="59.69" width="0.6096" layer="16"/>
+<wire x1="71.12" y1="55.88" x2="71.12" y2="58.42" width="0.6096" layer="16"/>
+<wire x1="38.1" y1="71.12" x2="49.53" y2="71.12" width="0.6096" layer="16"/>
+<wire x1="52.07" y1="59.69" x2="66.04" y2="59.69" width="0.6096" layer="16"/>
+<wire x1="66.675" y1="57.785" x2="68.58" y2="55.88" width="0.6096" layer="16"/>
+<wire x1="66.675" y1="59.055" x2="66.04" y2="59.69" width="0.6096" layer="16"/>
+<wire x1="66.675" y1="57.785" x2="66.675" y2="59.055" width="0.6096" layer="16"/>
+<wire x1="68.58" y1="55.88" x2="71.12" y2="55.88" width="0.6096" layer="16"/>
+<wire x1="36.83" y1="52.07" x2="36.83" y2="31.75" width="0.6096" layer="16"/>
 </signal>
 <signal name="S$13">
@@
 <wire x1="5.04" y1="41.91" x2="6.35" y2="41.91" width="0.6096" layer="16"/>
 </signal>
+<signal name="S$15">
+<contactref element="E$17" pad="10"/>
+<contactref element="E$41" pad="1"/>
+<wire x1="63.5" y1="53.34" x2="64.77" y2="53.34" width="0.6096" layer="16"/>
+<wire x1="64.77" y1="53.34" x2="66.04" y2="52.07" width="0.6096" layer="16"/>
+<wire x1="66.04" y1="52.07" x2="80.01" y2="52.07" width="0.6096" layer="16"/>
+<wire x1="80.01" y1="52.07" x2="81.28" y2="53.34" width="0.6096" layer="16"/>
+<wire x1="81.28" y1="53.34" x2="81.28" y2="58.42" width="0.6096" layer="16"/>
+<contactref element="E$11" pad="10"/>
+<contactref element="E$7" pad="10"/>
+<contactref element="E$5" pad="10"/>
+<wire x1="55.88" y1="53.34" x2="58.42" y2="53.34" width="0.6096" layer="16"/>
+<wire x1="58.42" y1="53.34" x2="60.96" y2="53.34" width="0.6096" layer="16"/>
+<wire x1="60.96" y1="53.34" x2="63.5" y2="53.34" width="0.6096" layer="16"/>
+</signal>
+<signal name="S$16">
+<contactref element="E$41" pad="2"/>
+<contactref element="E$16" pad="1"/>
+<wire x1="67.31" y1="53.34" x2="77.47" y2="53.34" width="0.6096" layer="16"/>
+<wire x1="77.47" y1="53.34" x2="78.74" y2="54.61" width="0.6096" layer="16"/>
+<wire x1="78.74" y1="54.61" x2="78.74" y2="58.42" width="0.6096" layer="16"/>
+<wire x1="64.77" y1="55.88" x2="67.31" y2="53.34" width="0.6096" layer="16"/>
+<wire x1="63.5" y1="55.88" x2="64.77" y2="55.88" width="0.6096" layer="16"/>
+<contactref element="E$10" pad="1"/>
+<contactref element="E$6" pad="1"/>
+<contactref element="E$4" pad="1"/>
+<wire x1="63.5" y1="55.88" x2="60.96" y2="55.88" width="0.6096" layer="16"/>
+<wire x1="60.96" y1="55.88" x2="58.42" y2="55.88" width="0.6096" layer="16"/>
+<wire x1="58.42" y1="55.88" x2="55.88" y2="55.88" width="0.6096" layer="16"/>
+</signal>
+<signal name="S$17">
+<contactref element="E$16" pad="8"/>
+<contactref element="E$41" pad="3"/>
+<wire x1="76.2" y1="58.42" x2="76.2" y2="71.12" width="0.6096" layer="16"/>
+<wire x1="76.2" y1="71.12" x2="73.66" y2="73.66" width="0.6096" layer="16"/>
+<wire x1="73.66" y1="73.66" x2="63.5" y2="73.66" width="0.6096" layer="16"/>
+<contactref element="E$10" pad="8"/>
+<contactref element="E$6" pad="8"/>
+<contactref element="E$4" pad="8"/>
+<wire x1="63.5" y1="73.66" x2="60.96" y2="73.66" width="0.6096" layer="16"/>
+<wire x1="60.96" y1="73.66" x2="58.42" y2="73.66" width="0.6096" layer="16"/>
+<wire x1="58.42" y1="73.66" x2="55.88" y2="73.66" width="0.6096" layer="16"/>
+</signal>
+<signal name="S$18">
+<contactref element="E$16" pad="2"/>
+<contactref element="E$41" pad="4"/>
+<wire x1="63.5" y1="58.42" x2="64.77" y2="58.42" width="0.6096" layer="16"/>
+<wire x1="72.39" y1="54.61" x2="73.66" y2="55.88" width="0.6096" layer="16"/>
+<wire x1="73.66" y1="55.88" x2="73.66" y2="58.42" width="0.6096" layer="16"/>
+<wire x1="64.77" y1="58.42" x2="68.58" y2="54.61" width="0.6096" layer="16"/>
+<wire x1="68.58" y1="54.61" x2="72.39" y2="54.61" width="0.6096" layer="16"/>
+<contactref element="E$10" pad="2"/>
+<contactref element="E$6" pad="2"/>
+<contactref element="E$4" pad="2"/>
+<wire x1="63.5" y1="58.42" x2="60.96" y2="58.42" width="0.6096" layer="16"/>
+<wire x1="60.96" y1="58.42" x2="58.42" y2="58.42" width="0.6096" layer="16"/>
+<wire x1="58.42" y1="58.42" x2="55.88" y2="58.42" width="0.6096" layer="16"/>
+</signal>
 </signals>
