File: Grbl_Esp32/src/custom/pcb/control board/controlBoard.brd (EAGLE design)
At the start: 41 parts

Commit message: controlBoard
Parts:
- moved E$41 1.27 mm to (76.2, 58.4)
Routing:
- net S$18: track 22.4 -> 23.7 mm
- net S$16: track 28.2 -> 28.8 mm
- net S$15: track 31.5 -> 32.1 mm
- net S$1: track 178.6 -> 179.1 mm
- net S$17: track 34.1 -> 34.6 mm
- net S$12: track 144.7 -> 145.2 mm
Changed lines of the file:
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@@
 <attribute name="VALUE" x="16.51" y="27.98" size="1.27" layer="27" ratio="10" rot="R90"/>
 </element>
-<element name="E$41" library="con-lsta" library_urn="urn:adsk.eagle:library:161" package="FE06" package3d_urn="urn:adsk.eagle:package:8191/1" value="" x="74.93" y="58.42" rot="R180">
-<attribute name="NAME" x="78.74" y="56.769" size="1.27" layer="25" ratio="10" rot="R180"/>
-<attribute name="VALUE" x="82.55" y="61.341" size="1.27" layer="27" ratio="10" rot="R180"/>
+<element name="E$41" library="con-lsta" library_urn="urn:adsk.eagle:library:161" package="FE06" package3d_urn="urn:adsk.eagle:package:8191/1" value="" x="76.2" y="58.42" rot="R180">
+<attribute name="NAME" x="80.01" y="56.769" size="1.27" layer="25" ratio="10" rot="R180"/>
+<attribute name="VALUE" x="83.82" y="61.341" size="1.27" layer="27" ratio="10" rot="R180"/>
 </element>
 <element name="E$42" library="con-lsta" library_urn="urn:adsk.eagle:library:161" package="FE07" package3d_urn="urn:adsk.eagle:package:8223/1" value="" x="81.28" y="38.1" rot="R90">
@@
 <contactref element="E$10" pad="3"/>
 <contactref element="E$6" pad="3"/>
-<wire x1="68.58" y1="58.42" x2="68.58" y2="59.69" width="0.6096" layer="16"/>
-<wire x1="68.58" y1="59.69" x2="67.31" y2="60.96" width="0.6096" layer="16"/>
+<wire x1="69.85" y1="58.42" x2="67.31" y2="60.96" width="0.6096" layer="16"/>
 <wire x1="67.31" y1="60.96" x2="63.5" y2="60.96" width="0.6096" layer="16"/>
 <wire x1="63.5" y1="60.96" x2="60.96" y2="60.96" width="0.6096" layer="16"/>
@@
 <wire x1="50.8" y1="69.85" x2="50.8" y2="60.96" width="0.6096" layer="16"/>
 <wire x1="50.8" y1="60.96" x2="52.07" y2="59.69" width="0.6096" layer="16"/>
-<wire x1="71.12" y1="55.88" x2="71.12" y2="58.42" width="0.6096" layer="16"/>
+<wire x1="72.39" y1="57.15" x2="72.39" y2="58.42" width="0.6096" layer="16"/>
 <wire x1="38.1" y1="71.12" x2="49.53" y2="71.12" width="0.6096" layer="16"/>
-<wire x1="52.07" y1="59.69" x2="66.04" y2="59.69" width="0.6096" layer="16"/>
-<wire x1="66.675" y1="57.785" x2="68.58" y2="55.88" width="0.6096" layer="16"/>
-<wire x1="66.675" y1="59.055" x2="66.04" y2="59.69" width="0.6096" layer="16"/>
-<wire x1="66.675" y1="57.785" x2="66.675" y2="59.055" width="0.6096" layer="16"/>
+<wire x1="66.04" y1="59.69" x2="52.07" y2="59.69" width="0.6096" layer="16"/>
 <wire x1="68.58" y1="55.88" x2="71.12" y2="55.88" width="0.6096" layer="16"/>
 <wire x1="36.83" y1="52.07" x2="36.83" y2="31.75" width="0.6096" layer="16"/>
+<wire x1="67.31" y1="58.42" x2="66.04" y2="59.69" width="0.6096" layer="16"/>
+<wire x1="68.58" y1="55.88" x2="67.31" y2="57.15" width="0.6096" layer="16"/>
+<wire x1="67.31" y1="57.15" x2="67.31" y2="58.42" width="0.6096" layer="16"/>
+<wire x1="71.12" y1="55.88" x2="72.39" y2="57.15" width="0.6096" layer="16"/>
 </signal>
 <signal name="S$13">
@@
 <wire x1="64.77" y1="53.34" x2="66.04" y2="52.07" width="0.6096" layer="16"/>
 <wire x1="66.04" y1="52.07" x2="80.01" y2="52.07" width="0.6096" layer="16"/>
-<wire x1="80.01" y1="52.07" x2="81.28" y2="53.34" width="0.6096" layer="16"/>
-<wire x1="81.28" y1="53.34" x2="81.28" y2="58.42" width="0.6096" layer="16"/>
+<wire x1="80.01" y1="52.07" x2="82.55" y2="54.61" width="0.6096" layer="16"/>
+<wire x1="82.55" y1="58.42" x2="82.55" y2="54.61" width="0.6096" layer="16"/>
 <contactref element="E$11" pad="10"/>
 <contactref element="E$7" pad="10"/>
@@
 <contactref element="E$16" pad="1"/>
 <wire x1="67.31" y1="53.34" x2="77.47" y2="53.34" width="0.6096" layer="16"/>
-<wire x1="77.47" y1="53.34" x2="78.74" y2="54.61" width="0.6096" layer="16"/>
-<wire x1="78.74" y1="54.61" x2="78.74" y2="58.42" width="0.6096" layer="16"/>
+<wire x1="77.47" y1="53.34" x2="80.01" y2="55.88" width="0.6096" layer="16"/>
+<wire x1="80.01" y1="58.42" x2="80.01" y2="55.88" width="0.6096" layer="16"/>
 <wire x1="64.77" y1="55.88" x2="67.31" y2="53.34" width="0.6096" layer="16"/>
 <wire x1="63.5" y1="55.88" x2="64.77" y2="55.88" width="0.6096" layer="16"/>
@@
 <contactref element="E$16" pad="8"/>
 <contactref element="E$41" pad="3"/>
-<wire x1="76.2" y1="58.42" x2="76.2" y2="71.12" width="0.6096" layer="16"/>
-<wire x1="76.2" y1="71.12" x2="73.66" y2="73.66" width="0.6096" layer="16"/>
+<wire x1="77.47" y1="69.85" x2="77.47" y2="58.42" width="0.6096" layer="16"/>
+<wire x1="77.47" y1="69.85" x2="73.66" y2="73.66" width="0.6096" layer="16"/>
 <wire x1="73.66" y1="73.66" x2="63.5" y2="73.66" width="0.6096" layer="16"/>
 <contactref element="E$10" pad="8"/>
@@
 <contactref element="E$41" pad="4"/>
 <wire x1="63.5" y1="58.42" x2="64.77" y2="58.42" width="0.6096" layer="16"/>
-<wire x1="72.39" y1="54.61" x2="73.66" y2="55.88" width="0.6096" layer="16"/>
-<wire x1="73.66" y1="55.88" x2="73.66" y2="58.42" width="0.6096" layer="16"/>
-<wire x1="64.77" y1="58.42" x2="68.58" y2="54.61" width="0.6096" layer="16"/>
-<wire x1="68.58" y1="54.61" x2="72.39" y2="54.61" width="0.6096" layer="16"/>
+<wire x1="74.93" y1="55.88" x2="73.66" y2="54.61" width="0.6096" layer="16"/>
+<wire x1="74.93" y1="58.42" x2="74.93" y2="55.88" width="0.6096" layer="16"/>
 <contactref element="E$10" pad="2"/>
 <contactref element="E$6" pad="2"/>
@@
 <wire x1="60.96" y1="58.42" x2="58.42" y2="58.42" width="0.6096" layer="16"/>
 <wire x1="58.42" y1="58.42" x2="55.88" y2="58.42" width="0.6096" layer="16"/>
+<wire x1="68.58" y1="54.61" x2="73.66" y2="54.61" width="0.6096" layer="16"/>
+<wire x1="64.77" y1="58.42" x2="68.58" y2="54.61" width="0.6096" layer="16"/>
 </signal>
 </signals>

Commit message: controlBoard
Parts:
- moved E$42 8.98 mm to (74.9, 44.5), turned to 180 degrees
Connections:
- new net S$19: E$11.9, E$17.9, E$42.3, E$5.9, E$7.9
- new net S$20: E$11.8, E$17.8, E$42.4, E$5.8, E$7.8
- net S$1: now also E$42.6
- net S$12: now also E$42.5
Routing:
- net S$12: track 145.2 -> 204.2 mm
- net S$1: track 179.1 -> 216.8 mm
- net S$19: track 0.00 -> 27.7 mm
- net S$20: track 0.00 -> 22.1 mm

Commit message: controlBoard
Routing:
- net S$17: track 34.6 -> 35.3 mm
Other:
- board text added: "Ahmed Sayed"
- board text added: "DR. MUSTAFA M. SHIPLE"
- board text added: "John Khalil"
- board text added: "Marwan Hesham"
Changed lines of the file:
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@@
 <board>
 <plain>
+<text x="44.45" y="34.29" size="1.778" layer="16" rot="MR90">Marwan Hesham</text>
+<text x="43.18" y="45.72" size="1.778" layer="16" rot="MR270">John Khalil</text>
+<text x="40.64" y="49.53" size="1.778" layer="16" rot="MR270">Ahmed Sayed</text>
+<text x="49.53" y="69.85" size="1.778" layer="16" rot="MR270">DR. MUSTAFA M. SHIPLE</text>
+<text x="17.78" y="67.31" size="1.778" layer="16" rot="MR0">John Khalil</text>
+<text x="74.93" y="64.77" size="1.778" layer="16" rot="MR0">Marwan
+Hesham</text>
 </plain>
 <attributes>
@@
 <contactref element="E$16" pad="8"/>
 <contactref element="E$41" pad="3"/>
-<wire x1="77.47" y1="69.85" x2="77.47" y2="58.42" width="0.6096" layer="16"/>
-<wire x1="77.47" y1="69.85" x2="73.66" y2="73.66" width="0.6096" layer="16"/>
-<wire x1="73.66" y1="73.66" x2="63.5" y2="73.66" width="0.6096" layer="16"/>
 <contactref element="E$10" pad="8"/>
 <contactref element="E$6" pad="8"/>
@@
 <wire x1="60.96" y1="73.66" x2="58.42" y2="73.66" width="0.6096" layer="16"/>
 <wire x1="58.42" y1="73.66" x2="55.88" y2="73.66" width="0.6096" layer="16"/>
+<wire x1="77.47" y1="58.42" x2="77.47" y2="71.12" width="0.6096" layer="16"/>
+<wire x1="77.47" y1="71.12" x2="74.93" y2="73.66" width="0.6096" layer="16"/>
+<wire x1="74.93" y1="73.66" x2="63.5" y2="73.66" width="0.6096" layer="16"/>
 </signal>
 <signal name="S$18">
@@
 </drawing>
 <compatibility>
+<note version="6.3" minversion="6.2.2" severity="warning">
+Since Version 6.2.2 text objects can contain more than one line,
+which will not be processed correctly with this version.
+</note>
 <note version="8.2" severity="warning">
 Since Version 8.2, EAGLE supports online libraries. The ids
