File: Grbl_Esp32/src/custom/pcb/plugin/plugin.brd (EAGLE design)
At the start: 21 parts

Commit message: plugin board
Parts:
- moved E$20 88.4 mm to (12.7, -6.35), turned to 270 degrees
- moved E$19 87.5 mm to (12.7, 3.81), turned to 270 degrees
Connections:
- removed net S$11: E$2.NC, E$6.NC, E$8.1
- removed net S$15: E$11.1, E$12.1, E$14.C
- removed net S$9: E$2.1, E$6.1, E$9.C
- net S$2: now also E$11.1, E$12.1, E$14.C, E$2.1, E$20.1, E$6.1, E$9.C
- net S$5: now also E$13.1, E$19.2, E$2.NC, E$6.NC, E$8.1
- net S$6: now also E$19.1
Routing:
- net S$5: track 24.0 -> 128.9 mm
- net S$2: track 9.07 -> 104.9 mm
- net S$6: track 52.1 -> 87.1 mm
- net S$11: track 25.3 -> 0.00 mm
- net S$9: track 9.07 -> 0.00 mm
- net S$15: track 9.07 -> 0.00 mm
- net S$8: track 33.2 -> 31.8 mm

Commit message: plugin board
Parts:
- added E$22: (no value), con-molex:70543-22
- added E$23: (no value), con-lstb:MA05-1
- added E$24: (no value), con-wago-508:W237-132
- added E$25, E$26, E$27, E$28: (no value), con-lstb:MA07-2
- moved E$19 1.27 mm to (11.4, 3.81)
- moved E$20 1.27 mm to (11.4, -6.35)
Connections:
- new net S$11: E$22.10, E$27.3, E$27.4
- new net S$15: E$22.11, E$27.5, E$27.6
- new net S$17: E$22.12, E$27.7, E$27.8
- new net S$20: E$22.13, E$27.10, E$27.9
- new net S$21: E$22.14, E$27.11, E$27.12
- new net S$22: E$22.15, E$27.13, E$27.14
- new net S$23: E$22.16, E$28.1, E$28.2
- new net S$24: E$22.17, E$28.3, E$28.4
- new net S$25: E$22.18, E$28.5, E$28.6
- new net S$26: E$22.19, E$28.7, E$28.8
- new net S$27: E$22.20, E$28.10, E$28.9
- new net S$28: E$22.21, E$28.11, E$28.12
- new net S$29: E$22.22, E$28.13, E$28.14
- new net S$30: E$1.A, E$22.6
- new net S$31: E$10.A, E$22.7
- new net S$32: E$15.A, E$22.8
- new net S$33: E$22.2, E$23.2
- new net S$34: E$22.3, E$23.3
- new net S$35: E$22.4, E$23.4
- new net S$36: E$22.5, E$23.5, E$25.10, E$25.12, E$25.14, E$25.2, E$25.4, E$25.6, E$25.8, E$26.10, E$26.12, E$26.14, E$26.2, E$26.4, E$26.6, E$26.8
- new net S$9: E$22.9, E$27.1, E$27.2
- net S$5: now also E$22.1, E$23.1, E$25.1, E$25.11, E$25.13, E$25.3, E$25.5, E$25.7, E$25.9, E$26.1, E$26.11, E$26.13, E$26.3, E$26.5, E$26.7, E$26.9
Routing:
- net S$5: track 128.9 -> 282.0 mm
- net S$36: track 0.00 -> 51.3 mm
- net S$32: track 0.00 -> 21.9 mm
- net S$30: track 0.00 -> 17.0 mm
- net S$31: track 0.00 -> 6.88 mm
- net S$9: track 0.00 -> 6.35 mm
- net S$29: track 0.00 -> 6.35 mm
- net S$28: track 0.00 -> 6.35 mm
- net S$27: track 0.00 -> 6.35 mm
- net S$26: track 0.00 -> 6.35 mm
- net S$25: track 0.00 -> 6.35 mm
- net S$24: track 0.00 -> 6.35 mm
- net S$23: track 0.00 -> 6.35 mm
- net S$22: track 0.00 -> 6.35 mm
- net S$21: track 0.00 -> 6.35 mm
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
Commit message: plugin board
Parts:
- moved E$24 22.2 mm to (33.0, -11.4), turned to 0 degrees
Connections:
- removed net S$5: E$13.1, E$19.2, E$2.NC, E$22.1, E$23.1, E$25.1, E$25.11, E$25.13, E$25.3, E$25.5, E$25.7, E$25.9, E$26.1, E$26.11, E$26.13, E$26.3, E$26.5, E$26.7, E$26.9, E$3.NC, E$4.NC, E$5.1, E$6.NC, E$8.1
- new net S$39: E$22.5, E$23.5, E$24.1, E$25.1, E$25.11, E$25.13, E$25.3, E$25.5, E$25.7, E$25.9, E$26.1, E$26.11, E$26.13, E$26.3, E$26.5, E$26.7, E$26.9
- net S$36: now also E$13.1, E$19.2, E$2.NC, E$22.1, E$23.1, E$24.2, E$3.NC, E$4.NC, E$5.1, E$6.NC, E$8.1; no longer E$22.5, E$23.5
Routing:
- net S$36: track 51.3 -> 334.8 mm
- net S$5: track 282.0 -> 0.00 mm
- net S$39: track 0.00 -> 56.4 mm

Commit message: plugin board
Parts:
- added E$30, E$31, E$32: (no value), con-lsta:FE06
Connections:
- removed net S$39: E$22.5, E$23.5, E$24.1, E$25.1, E$25.11, E$25.13, E$25.3, E$25.5, E$25.7, E$25.9, E$26.1, E$26.11, E$26.13, E$26.3, E$26.5, E$26.7, E$26.9
- new net S$40: E$30.4, E$31.4, E$32.4
- new net S$41: E$30.3, E$31.3, E$32.3
- new net S$43: E$20.2, E$30.1, E$31.1, E$32.1
- net S$2: now also E$22.5, E$23.5, E$24.1, E$25.1, E$25.11, E$25.13, E$25.3, E$25.5, E$25.7, E$25.9, E$26.1, E$26.11, E$26.13, E$26.3, E$26.5, E$26.7, E$26.9, E$30.2, E$31.2, E$32.2
- net S$36: now also E$30.5, E$30.6, E$31.5, E$31.6, E$32.5, E$32.6
Routing:
- net S$2: track 105.0 -> 216.7 mm
- net S$36: track 334.8 -> 427.3 mm
- net S$43: track 0.00 -> 80.1 mm
- net S$39: track 56.4 -> 0.00 mm
- net S$41: track 0.00 -> 7.62 mm
- net S$40: track 0.00 -> 7.62 mm
Other:
- board text added: "John Khalil"
- board text added: "Marwan Hesham"
Changed lines of the file:
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@@
 <board>
 <plain>
+<text x="67.31" y="11.43" size="1.778" layer="16" rot="MR270">John Khalil</text>
+<text x="69.85" y="17.78" size="1.778" layer="16" rot="MR270">Marwan Hesham</text>
+<text x="33.02" y="-27.94" size="1.778" layer="16" rot="MR180">Marwan Hesham</text>
+<text x="38.1" y="-22.86" size="1.778" layer="16" rot="MR180">John Khalil</text>
 </plain>
 <attributes>
@@
 <attribute name="VALUE" x="29.21" y="-18.415" size="1.27" layer="27" ratio="10"/>
 </element>
+<element name="E$30" library="con-lsta" library_urn="urn:adsk.eagle:library:161" package="FE06" package3d_urn="urn:adsk.eagle:package:8191/1" value="" x="66.04" y="-31.75" rot="R90">
+<attribute name="NAME" x="64.389" y="-35.56" size="1.27" layer="25" ratio="10" rot="R90"/>
+<attribute name="VALUE" x="68.961" y="-39.37" size="1.27" layer="27" ratio="10" rot="R90"/>
+</element>
+<element name="E$31" library="con-lsta" library_urn="urn:adsk.eagle:library:161" package="FE06" package3d_urn="urn:adsk.eagle:package:8191/1" value="" x="62.23" y="-31.75" rot="R90">
+<attribute name="NAME" x="60.579" y="-35.56" size="1.27" layer="25" ratio="10" rot="R90"/>
+<attribute name="VALUE" x="65.151" y="-39.37" size="1.27" layer="27" ratio="10" rot="R90"/>
+</element>
+<element name="E$32" library="con-lsta" library_urn="urn:adsk.eagle:library:161" package="FE06" package3d_urn="urn:adsk.eagle:package:8191/1" value="" x="58.42" y="-31.75" rot="R90">
+<attribute name="NAME" x="56.769" y="-35.56" size="1.27" layer="25" ratio="10" rot="R90"/>
+<attribute name="VALUE" x="61.341" y="-39.37" size="1.27" layer="27" ratio="10" rot="R90"/>
+</element>
 </elements>
 <signals>
@@
 <wire x1="40.64" y1="13.97" x2="40.64" y2="6.35" width="0.6096" layer="16"/>
 <contactref element="E$20" pad="1"/>
-<wire x1="10.795" y1="-3.81" x2="10.795" y2="-1.905" width="0.6096" layer="16"/>
-<wire x1="10.795" y1="-1.905" x2="11.43" y2="-1.27" width="0.6096" layer="16"/>
-<wire x1="12.7" y1="-1.27" x2="11.43" y2="-1.27" width="0.6096" layer="16"/>
-<wire x1="12.7" y1="-1.27" x2="13.97" y2="0" width="0.6096" layer="16"/>
 <wire x1="16.51" y1="5.08" x2="21.59" y2="5.08" width="0.6096" layer="16"/>
 <wire x1="21.59" y1="5.08" x2="22.86" y2="6.35" width="0.6096" layer="16"/>
-<wire x1="13.97" y1="0" x2="13.97" y2="2.54" width="0.6096" layer="16"/>
 <wire x1="13.97" y1="2.54" x2="16.51" y2="5.08" width="0.6096" layer="16"/>
-</signal>
-<signal name="S$4">
-<contactref element="E$3" pad="2"/>
-<contactref element="E$4" pad="2"/>
-<contactref element="E$7" pad="A"/>
-<contactref element="E$5" pad="3"/>
-<wire x1="13.05" y1="19.97" x2="13.685" y2="20.605" width="2.54" layer="16"/>
-<wire x1="13.685" y1="20.605" x2="14.05" y2="20.97" width="1.27" layer="16"/>
-<wire x1="14.05" y1="20.97" x2="14.05" y2="21.35" width="2.54" layer="16"/>
-<wire x1="15.24" y1="13.97" x2="15.24" y2="11.43" width="0.6096" layer="16"/>
-<wire x1="15.24" y1="13.97" x2="13.97" y2="13.97" width="0.6096" layer="16"/>
-<wire x1="13.97" y1="13.97" x2="13.05" y2="14.89" width="0.6096" layer="16"/>
-<wire x1="13.05" y1="14.89" x2="13.05" y2="19.97" width="0.6096" layer="16"/>
-</signal>
-<signal name="S$39">
 <contactref element="E$26" pad="13"/>
 <contactref element="E$26" pad="11"/>
@@
 <wire x1="30.48" y1="-12.065" x2="27.94" y2="-12.065" width="0.6096" layer="16"/>
 <wire x1="27.94" y1="-12.065" x2="27.94" y2="-8.89" width="0.6096" layer="16"/>
+<wire x1="10.795" y1="-3.81" x2="13.97" y2="-3.81" width="0.6096" layer="16"/>
+<wire x1="13.97" y1="-5.08" x2="15.24" y2="-6.35" width="0.6096" layer="16"/>
+<wire x1="15.24" y1="-11.43" x2="17.78" y2="-13.97" width="0.6096" layer="16"/>
+<wire x1="17.78" y1="-13.97" x2="27.94" y2="-13.97" width="0.6096" layer="16"/>
+<wire x1="15.24" y1="-6.35" x2="15.24" y2="-11.43" width="0.6096" layer="16"/>
+<wire x1="13.97" y1="2.54" x2="13.97" y2="-3.81" width="0.6096" layer="16"/>
+<wire x1="13.97" y1="-3.81" x2="13.97" y2="-5.08" width="0.6096" layer="16"/>
+<contactref element="E$31" pad="2"/>
+<contactref element="E$32" pad="2"/>
+<contactref element="E$30" pad="2"/>
+<wire x1="62.23" y1="-35.56" x2="58.42" y2="-35.56" width="0.6096" layer="16"/>
+<wire x1="66.04" y1="-35.56" x2="62.23" y2="-35.56" width="0.6096" layer="16"/>
+<wire x1="69.85" y1="-35.56" x2="71.12" y2="-34.29" width="0.6096" layer="16"/>
+<wire x1="71.12" y1="-34.29" x2="71.12" y2="-15.24" width="0.6096" layer="16"/>
+<wire x1="66.04" y1="-35.56" x2="69.85" y2="-35.56" width="0.6096" layer="16"/>
+</signal>
+<signal name="S$4">
+<contactref element="E$3" pad="2"/>
+<contactref element="E$4" pad="2"/>
+<contactref element="E$7" pad="A"/>
+<contactref element="E$5" pad="3"/>
+<wire x1="13.05" y1="19.97" x2="13.685" y2="20.605" width="2.54" layer="16"/>
+<wire x1="13.685" y1="20.605" x2="14.05" y2="20.97" width="1.27" layer="16"/>
+<wire x1="14.05" y1="20.97" x2="14.05" y2="21.35" width="2.54" layer="16"/>
+<wire x1="15.24" y1="13.97" x2="15.24" y2="11.43" width="0.6096" layer="16"/>
+<wire x1="15.24" y1="13.97" x2="13.97" y2="13.97" width="0.6096" layer="16"/>
+<wire x1="13.97" y1="13.97" x2="13.05" y2="14.89" width="0.6096" layer="16"/>
+<wire x1="13.05" y1="14.89" x2="13.05" y2="19.97" width="0.6096" layer="16"/>
 </signal>
 <signal name="S$6">
@@
 <wire x1="35.56" y1="-12.065" x2="35.56" y2="-12.7" width="0.6096" layer="16"/>
 <wire x1="35.56" y1="-12.7" x2="38.1" y2="-12.7" width="0.6096" layer="16"/>
+<contactref element="E$31" pad="5"/>
+<contactref element="E$32" pad="5"/>
+<contactref element="E$30" pad="5"/>
+<wire x1="62.23" y1="-27.94" x2="58.42" y2="-27.94" width="0.6096" layer="16"/>
+<wire x1="66.04" y1="-27.94" x2="62.23" y2="-27.94" width="0.6096" layer="16"/>
+<contactref element="E$31" pad="6"/>
+<contactref element="E$32" pad="6"/>
+<contactref element="E$30" pad="6"/>
+<wire x1="62.23" y1="-25.4" x2="58.42" y2="-25.4" width="0.6096" layer="16"/>
+<wire x1="66.04" y1="-25.4" x2="62.23" y2="-25.4" width="0.6096" layer="16"/>
+<wire x1="62.23" y1="-25.4" x2="62.23" y2="-27.94" width="0.6096" layer="16"/>
+<wire x1="10.795" y1="1.27" x2="8.89" y2="1.27" width="0.6096" layer="16"/>
+<wire x1="8.89" y1="1.27" x2="7.62" y2="0" width="0.6096" layer="16"/>
+<wire x1="7.62" y1="0" x2="7.62" y2="-5.08" width="0.6096" layer="16"/>
+<wire x1="7.62" y1="-5.08" x2="8.89" y2="-6.35" width="0.6096" layer="16"/>
+<wire x1="8.89" y1="-6.35" x2="12.7" y2="-6.35" width="0.6096" layer="16"/>
+<wire x1="12.7" y1="-6.35" x2="13.97" y2="-7.62" width="0.6096" layer="16"/>
+<wire x1="13.97" y1="-7.62" x2="13.97" y2="-12.7" width="0.6096" layer="16"/>
+<wire x1="13.97" y1="-12.7" x2="16.51" y2="-15.24" width="0.6096" layer="16"/>
+<wire x1="16.51" y1="-15.24" x2="26.67" y2="-15.24" width="0.6096" layer="16"/>
+<wire x1="26.67" y1="-15.24" x2="29.21" y2="-17.78" width="0.6096" layer="16"/>
+<wire x1="57.15" y1="-17.78" x2="58.42" y2="-19.05" width="0.6096" layer="16"/>
+<wire x1="58.42" y1="-19.05" x2="58.42" y2="-25.4" width="0.6096" layer="16"/>
+<wire x1="29.21" y1="-17.78" x2="57.15" y2="-17.78" width="0.6096" layer="16"/>
 </signal>
 <signal name="S$30">
@@
 <wire x1="35.56" y1="-2.54" x2="39.37" y2="1.27" width="0.6096" layer="16"/>
 </signal>
+<signal name="S$40">
+<contactref element="E$31" pad="4"/>
+<contactref element="E$32" pad="4"/>
+<contactref element="E$30" pad="4"/>
+<wire x1="62.23" y1="-30.48" x2="58.42" y2="-30.48" width="0.6096" layer="16"/>
+<wire x1="66.04" y1="-30.48" x2="62.23" y2="-30.48" width="0.6096" layer="16"/>
+</signal>
+<signal name="S$41">
+<contactref element="E$31" pad="3"/>
+<contactref element="E$32" pad="3"/>
+<contactref element="E$30" pad="3"/>
+<wire x1="62.23" y1="-33.02" x2="58.42" y2="-33.02" width="0.6096" layer="16"/>
+<wire x1="66.04" y1="-33.02" x2="62.23" y2="-33.02" width="0.6096" layer="16"/>
+</signal>
+<signal name="S$43">
+<contactref element="E$31" pad="1"/>
+<contactref element="E$32" pad="1"/>
+<contactref element="E$30" pad="1"/>
+<wire x1="62.23" y1="-38.1" x2="58.42" y2="-38.1" width="0.6096" layer="16"/>
+<wire x1="63.5" y1="-38.1" x2="62.23" y2="-38.1" width="0.6096" layer="16"/>
+<wire x1="66.04" y1="-38.1" x2="62.23" y2="-38.1" width="0.6096" layer="16"/>
+<contactref element="E$20" pad="2"/>
+<wire x1="10.795" y1="-8.89" x2="10.795" y2="-13.335" width="0.6096" layer="16"/>
+<wire x1="24.13" y1="-17.78" x2="26.67" y2="-20.32" width="0.6096" layer="16"/>
+<wire x1="53.34" y1="-20.32" x2="54.61" y2="-21.59" width="0.6096" layer="16"/>
+<wire x1="54.61" y1="-21.59" x2="54.61" y2="-36.83" width="0.6096" layer="16"/>
+<wire x1="54.61" y1="-36.83" x2="55.88" y2="-38.1" width="0.6096" layer="16"/>
+<wire x1="55.88" y1="-38.1" x2="58.42" y2="-38.1" width="0.6096" layer="16"/>
+<wire x1="10.795" y1="-13.335" x2="15.24" y2="-17.78" width="0.6096" layer="16"/>
+<wire x1="15.24" y1="-17.78" x2="24.13" y2="-17.78" width="0.6096" layer="16"/>
+<wire x1="26.67" y1="-20.32" x2="53.34" y2="-20.32" width="0.6096" layer="16"/>
+</signal>
 </signals>
